File: kohlbecker/BB816/hardware/breakout/breakout.kicad_pcb (KiCad board)
At the start: 4 copper layers, 152.4 x 64.8 mm, 32 parts, among them J1 Barrel_Jack_Switch, J2 Conn_02x40_Odd_Even, J3 Conn_02x18_Odd_Even, U7 74AHC125, U9 74HC74, X1 8MHz

Commit message: New pcb
Parts:
- removed R11: 3.3k, Resistor_THT:R_Axial_DIN0207_L6.3mm_D2.5mm_P7.62mm_Horizontal
- removed R12: 100k, Resistor_THT:R_Axial_DIN0207_L6.3mm_D2.5mm_P7.62mm_Horizontal
- removed TP1: 8MHz, TestPoint:TestPoint_THTPad_D1.5mm_Drill0.7mm
- removed TP10: READ_CLK, TestPoint:TestPoint_THTPad_D1.5mm_Drill0.7mm
- removed TP11: WRITE_CLK, TestPoint:TestPoint_THTPad_D1.5mm_Drill0.7mm
- removed TP12: RDY_REG, TestPoint:TestPoint_THTPad_D1.5mm_Drill0.7mm
- removed TP13: ~{RDY_REG}, TestPoint:TestPoint_THTPad_D1.5mm_Drill0.7mm
- removed TP14: B_~{OE}, TestPoint:TestPoint_THTPad_D1.5mm_Drill0.7mm
- removed TP15: ~{BE}, TestPoint:TestPoint_THTPad_D1.5mm_Drill0.7mm
- removed TP2: RDY⎒, TestPoint:TestPoint_THTPad_D1.5mm_Drill0.7mm
- removed TP3: VDA, TestPoint:TestPoint_THTPad_D1.5mm_Drill0.7mm
- removed TP4: VPA, TestPoint:TestPoint_THTPad_D1.5mm_Drill0.7mm
- removed TP5: MX, TestPoint:TestPoint_THTPad_D1.5mm_Drill0.7mm
- removed TP6: CLK-, TestPoint:TestPoint_THTPad_D1.5mm_Drill0.7mm
- removed TP7: CLK+, TestPoint:TestPoint_THTPad_D1.5mm_Drill0.7mm
- removed TP8: BUFFER_CLK, TestPoint:TestPoint_THTPad_D1.5mm_Drill0.7mm
- removed TP9: ~{READ_CLK}, TestPoint:TestPoint_THTPad_D1.5mm_Drill0.7mm
- removed U7: 74AHC125, Package_DIP:DIP-14_W7.62mm
- removed U9: 74HC74, Package_DIP:DIP-14_W7.62mm
- removed X1: 8MHz, Oscillator:Oscillator_DIP-8
- added C10: 100nF, Capacitor_THT:C_Disc_D3.4mm_W2.1mm_P2.50mm, F.Cu at (113.2, 96.8)
- added C11: 100nF, Capacitor_THT:C_Disc_D3.4mm_W2.1mm_P2.50mm, F.Cu at (118.9, 78.5)
- added C12: 100nF, Capacitor_THT:C_Disc_D3.4mm_W2.1mm_P2.50mm, F.Cu at (118.9, 82.2)
- added C13: 100nF, Capacitor_THT:C_Disc_D3.4mm_W2.1mm_P2.50mm, F.Cu at (118.9, 85.8)
- added C14: 100nF, Capacitor_THT:C_Disc_D3.4mm_W2.1mm_P2.50mm, F.Cu at (132.8, 91.5)
- added C15: 100nF, Capacitor_THT:C_Disc_D3.4mm_W2.1mm_P2.50mm, F.Cu at (129.8, 71.2)
- added C5: 100nF, Capacitor_THT:C_Disc_D3.4mm_W2.1mm_P2.50mm, F.Cu at (113.2, 78.5)
- added C6: 100nF, Capacitor_THT:C_Disc_D3.4mm_W2.1mm_P2.50mm, F.Cu at (113.2, 82.2)
- added C7: 100nF, Capacitor_THT:C_Disc_D3.4mm_W2.1mm_P2.50mm, F.Cu at (113.2, 85.8)
- added C8: 100nF, Capacitor_THT:C_Disc_D3.4mm_W2.1mm_P2.50mm, F.Cu at (113.2, 89.5)
- added C9: 100nF, Capacitor_THT:C_Disc_D3.4mm_W2.1mm_P2.50mm, F.Cu at (113.2, 93.1)
- added J4: I/O, Connector_PinHeader_2.54mm:PinHeader_2x08_P2.54mm_Vertical, F.Cu at (70.4, 71.0)
- added J5: Decoder Output, Connector_PinHeader_2.54mm:PinHeader_2x08_P2.54mm_Vertical, F.Cu at (40.4, 71.5)
- added J7: VP_REWR, Connector_PinHeader_2.54mm:PinHeader_2x05_P2.54mm_Vertical, F.Cu at (142.2, 121.8)
- added U1: 74LS04, Package_DIP:DIP-14_W7.62mm, F.Cu at (67.0, 98.4)
- added U12: 74LS138, Package_DIP:DIP-16_W7.62mm, F.Cu at (68.4, 83.6)
- added U14: AT28C256-15PC, Socket:DIP_Socket-28_W11.9_W12.7_W15.24_W17.78_W18.5_3M_228-1277-00-0602J, F.Cu at (135.5, 112.5)
- added U15: AS6C4008-55PCN, Package_DIP:DIP-32_W15.24mm, F.Cu at (129.9, 88.9)
- added U2: 74LS32, Package_DIP:DIP-14_W7.62mm, F.Cu at (66.9, 117.6)
- added U3: 74LS32, Package_DIP:DIP-14_W7.62mm, F.Cu at (45.9, 101.1)
- added U5: 74LS08, Package_DIP:DIP-14_W7.62mm, F.Cu at (28.4, 114.1)
- added U6: 74LS138, Package_DIP:DIP-16_W7.62mm, F.Cu at (91.4, 88.9)
- added U8: 74LS138, Package_DIP:DIP-16_W7.62mm, F.Cu at (106.7, 111.5)
- moved C4 45.9 mm to (42.0, 53.6), turned to 90 degrees
- moved R6 21.8 mm to (38.1, 52.4)
- moved C1 21.8 mm to (24.1, 55.0)
- moved C3 21.8 mm to (30.5, 57.8)
- moved D1 21.8 mm to (35.6, 57.8)
Connections:
- J3 pad 11: /A4 -> /AA4
- J3 pad 13: /A3 -> /AA3
- J3 pad 15: /A2 -> /AA2
- J3 pad 17: /A1 -> /AA1
Routing:
- net /~{VP}: track 0.00 -> 58.1 mm
- net /D3: track 0.00 -> 34.4 mm
- net /D4: track 0.00 -> 32.6 mm
- net /D5: track 0.00 -> 32.3 mm
- net /D6: track 0.00 -> 30.5 mm
- net /D7: track 0.00 -> 30.2 mm
- net /D2: track 0.00 -> 22.6 mm
- net /D0: track 0.00 -> 20.5 mm
- net /D1: track 0.00 -> 18.4 mm
- net /AA4: track 0.00 -> 5.26 mm
- net /AA3: track 0.00 -> 5.26 mm
- net /AA2: track 0.00 -> 5.26 mm
- net /AA1: track 0.00 -> 5.26 mm
Other:
- board text removed: "74HC74"
- board text removed: "8MHz"
