File: kohlbecker/BB816/hardware/breakout/breakout.kicad_sch (KiCad schematic)
At the start: 81 parts, among them J1 Barrel_Jack_Switch, J2 Conn_02x40_Odd_Even, J3 Conn_02x18_Odd_Even, SW1 RESET, U1 74AHC74, U10 74AHCT245, U11 74AHC573, U12 74AHC32, U13 74AHC02, U14 74HC74, U15 74AC10, U16 DS1035-10, U2 74AHC00, U3 74AC112, U4 W65C816SxP, U5 74AHC32, U6 74AHC32, U7 74AHC125, U8 DS1813-5, U9 74HC74, X1 8MHz

Commit message: Ready update schematic with added components to breakout
Parts:
- removed C10, C11, C12, C13, C14, C15, C16, C17, C18, C19, C5, C6, C7, C8, C9: 100n, Capacitor_THT:C_Disc_D3.4mm_W2.1mm_P2.50mm, symbol Device:C_Small
- removed D2: 1N5817, Diode_THT:D_DO-41_SOD81_P7.62mm_Horizontal, symbol Diode:1N5817
- removed R1, R17, R2, R3, R5: 3.3k, Resistor_THT:R_Axial_DIN0207_L6.3mm_D2.5mm_P7.62mm_Horizontal, symbol Device:R_Small
- removed R10, R7, R8, R9: 0R, BB816:0R_Jumper_R_Axial_DIN0207_L6.3mm_D2.5mm_P7.62mm_Horizontal, symbol Device:R_Small
- removed R13, R14, R15, R4: 100k, Resistor_THT:R_Axial_DIN0207_L6.3mm_D2.5mm_P7.62mm_Horizontal, symbol Device:R_Small
- removed R16: 1k, Resistor_THT:R_Axial_DIN0207_L6.3mm_D2.5mm_P7.62mm_Horizontal, symbol Device:R_Small
- removed RN1, RN2, RN3, RN4, RN5: 100k, Resistor_THT:R_Array_SIP9, symbol Device:R_Network08
- removed SW1: RESET, Button_Switch_THT:SW_PUSH_6mm, symbol Switch:SW_Push
- removed TP10: READ_CLK, TestPoint:TestPoint_THTPad_D1.5mm_Drill0.7mm, symbol Connector:TestPoint
- removed TP11: WRITE_CLK, TestPoint:TestPoint_THTPad_D1.5mm_Drill0.7mm, symbol Connector:TestPoint
- removed TP12: RDY_REG, TestPoint:TestPoint_THTPad_D1.5mm_Drill0.7mm, symbol Connector:TestPoint
- removed TP13: ~{RDY_REG}, TestPoint:TestPoint_THTPad_D1.5mm_Drill0.7mm, symbol Connector:TestPoint
- removed TP14: B_~{OE}, TestPoint:TestPoint_THTPad_D1.5mm_Drill0.7mm, symbol Connector:TestPoint
- removed TP15: ~{BE}, TestPoint:TestPoint_THTPad_D1.5mm_Drill0.7mm, symbol Connector:TestPoint
- removed TP8: BUFFER_CLK, TestPoint:TestPoint_THTPad_D1.5mm_Drill0.7mm, symbol Connector:TestPoint
- removed TP9: ~{READ_CLK}, TestPoint:TestPoint_THTPad_D1.5mm_Drill0.7mm, symbol Connector:TestPoint
- removed U1: 74AHC74, Package_DIP:DIP-14_W7.62mm, symbol 74xx:74LS74
- removed U10: 74AHCT245, Package_DIP:DIP-20_W7.62mm, symbol BB816:74AC245
- removed U11: 74AHC573, Package_DIP:DIP-20_W7.62mm, symbol 74xx:74LS573
- removed U12, U6: 74AHC32, Package_DIP:DIP-14_W7.62mm, symbol 74xx:74LS32
- removed U13: 74AHC02, Package_DIP:DIP-14_W7.62mm, symbol 74xx:74LS02
- removed U14: 74HC74, Package_DIP:DIP-14_W7.62mm, symbol 74xx:74LS74
- removed U15: 74AC10, Package_DIP:DIP-14_W7.62mm, symbol 74xx:74LS10
- removed U16: DS1035-10, Package_DIP:DIP-8_W7.62mm, symbol BB816:DS1035-10
- removed U2: 74AHC00, Package_DIP:DIP-14_W7.62mm, symbol 74xx:74HC00
- removed U3: 74AC112, Package_DIP:DIP-16_W7.62mm, symbol 74xx:74LS112
- removed U4: W65C816SxP, Package_DIP:DIP-40_W15.24mm, symbol BB816:W65C816SxP
- removed unit 3 of U5
- removed unit 2 of U5
- removed unit 1 of U5
- removed unit 4 of U5
- removed unit 4 of U7
- removed unit 1 of U7
- removed unit 2 of U7
- removed U8: DS1813-5, Package_TO_SOT_THT:TO-92_Inline, symbol BB816:DS1813
- added C10, C11, C12, C13, C14, C15, C5, C6, C7, C8, C9: 100nF, symbol Device:C
- added J4: Conn_02x8_Odd_Even, Connector_PinHeader_2.54mm:PinHeader_2x16_P2.54mm_Vertical, symbol Connector_Generic:Conn_02x08_Odd_Even
- added U1: 74LS04, Package_DIP:DIP-14_W7.62mm, symbol 74xx:74LS04
- added U10, U4: 74LS08, Package_DIP:DIP-14_W7.62mm, symbol 74xx:74LS08
- added U12, U6, U8: 74LS138, Package_DIP:DIP-16_W7.62mm, symbol 74xx:74LS138
- added U14: AT28C256-15PC, Socket:DIP_Socket-28_W11.9_W12.7_W15.24_W17.78_W18.5_3M_228-1277-00-0602J, symbol Memory_EEPROM:28C256
- added U15: AS6C4008-55PCN, Package_DIP:DIP-32_W15.24mm, symbol Memory_RAM:AS6C4008-55PCN
- added U2, U3: 74LS32, Package_DIP:DIP-14_W7.62mm, symbol 74xx:74LS32
- added X2: 16MHz, Oscillator:Oscillator_DIP-8, symbol Oscillator:CXO_DIP8
- TP1: value 8MHz -> ~{MEG0}
- TP2: value RDY⎒ -> ~{MEG0_LO}
- TP3: value VDA -> MEG0_HI
- TP4: value VPA -> ~{BANK0_HI}
- TP5: value MX -> ~{BANK0_LO}
- TP6: value CLK- -> ~{ROM_OE}
- TP7: value CLK+ -> ~{PAGE1}
- U5: value 74AHC32 -> 74LS32
Connections:
- net A0: now also U14.10 (A0), U15.12 (A0)
- net A1: now also U14.9 (A1), U15.11 (A1)
- net A10: now also U14.21 (A10), U15.23 (A10), U8.3 (A2)
- net A11: now also U14.23 (A11), U15.25 (A11), U6.1 (A0), U8.5 (E2)
- net A12: now also U14.2 (A12), U15.4 (A12), U6.2 (A1)
- net A13: now also U14.26 (A13), U15.28 (A13), U6.3 (A2)
- net A14: now also U14.1 (A14), U15.3 (A14), U6.5 (E2)
- net A15: now also U1.5, U15.31 (A15), U3.10
- net A16: now also U15.2 (A16)
- net A17: now also U15.30 (A17)
- net A18: now also U15.1 (A18)
- net A19: now also U10.2, U2.13
- net A2: now also U14.8 (A2), U15.10 (A2)
- net A20: now also U2.5
- net A21: now also U2.4
- net A22: now also U2.2
- net A23: now also U2.1
- net A3: now also U14.7 (A3), U15.9 (A3)
- net A4: now also U14.6 (A4), U15.8 (A4)
- net A5: now also U12.1 (A0), U14.5 (A5), U15.7 (A5)
- net A6: now also U12.2 (A1), U14.4 (A6), U15.6 (A6)
- net A7: now also U12.3 (A2), U14.3 (A7), U15.5 (A7)
- net A8: now also U14.25 (A8), U15.27 (A8), U8.1 (A0)
- net A9: now also U14.24 (A9), U15.26 (A9), U8.2 (A1)
- net CLK: no longer U9.3 (C)
- net D0: now also U14.11 (D0), U15.13 (DQ0)
- net D1: now also U14.12 (D1), U15.14 (DQ1)
- net D2: now also U14.13 (D2), U15.15 (DQ2)
- net D3: now also U14.15 (D3), U15.17 (DQ3)
- net D4: now also U14.16 (D4), U15.18 (DQ4)
- net D5: now also U14.17 (D5), U15.19 (DQ5)
- net D6: now also U14.18 (D6), U15.20 (DQ6)
- net D7: now also U14.19 (D7), U15.21 (DQ7)
- net E: now also X1.1 (EN), U1.13, U1.3, U4.2
- net GND: now also C10.2, C11.2, C12.2, C13.2, C14.2, C15.2, C5.2, C6.2, C7.2, C8.2, C9.2, J4.10 (Pin_10), J4.12 (Pin_12), J4.14 (Pin_14), J4.16 (Pin_16), J4.2 (Pin_2), J4.4 (Pin_4), J4.6 (Pin_6), J4.8 (Pin_8), U1.7 (GND), U14.14 (GND), U15.16 (VSS), U2.7 (GND), U3.7 (GND), U4.7 (GND), X2.4 (GND)
- net VCC: now also C10.1, C11.1, C12.1, C13.1, C14.1, C15.1, C5.1, C6.1, C7.1, C8.1, C9.1, U1.14 (VCC), U12.16 (VCC), U12.6 (E3), U14.28 (VCC), U15.32 (VCC), U2.14 (VCC), U3.14 (VCC), U4.14 (VCC), U6.16 (VCC), U6.6 (E3), U8.16 (VCC), U8.6 (E3), X2.8 (Vcc); no longer U9.4 (~{S})
- net ~{BANK0}: now also U3.5, U3.9
- net ~{MR}⎒: no longer U9.1 (~{R}), U9.2 (D)
- net ~{WR}: now also U14.27 (~{WE}), U15.29 (WE#)
- net 8MHz renamed 16MHz
- net 16MHz: now also X2.5 (OUT); no longer TP1.1
- net CLK+ renamed ~{PAGE1}
- net ~{PAGE1}: now also U1.11, U12.5 (E2), U8.14 (O1)
- net CLK- renamed ~{ROM_OE}
- net ~{ROM_OE}: now also U14.22 (~{OE}), U3.3
- net MX renamed ~{BANK0_LO}
- net ~{BANK0_LO}: now also U3.8, U6.4 (E1)
- net RDY⎒ renamed ~{MEGO_LO}
- net VDA renamed MEGO_HI
- net VPA renamed ~{BANK0_HI}
- net ~{BANK0_HI}: now also U1.9, U14.20 (~{CS}), U3.2, U3.6
- new net: U1.6, U3.4
- new net: U1.8, U4.1
- new net: U15.24 (OE#), U3.11
- new net: U6.15 (O0), U8.4 (E1)
- new net: U2.10, U2.6
- new net: U2.3, U2.9
- new net: U3.12, U4.3
- new net: U1.10, U3.13
- new net: U1.4, U3.1
- new net: U1.12, X2.1 (EN)
- new net: U12.4 (E1), U12.8 (GND)
- new net MEG0: U1.2, U10.1
- new net MEG0_HI: U10.3
- new net ~{0x00}: J4.1 (Pin_1), U12.15 (O0)
- new net ~{0x20}: J4.3 (Pin_3), U12.14 (O1)
- new net ~{0x40}: J4.5 (Pin_5)
- new net ~{0x60}: J4.7 (Pin_7), U12.12 (O3)
- new net ~{0x80}: J4.9 (Pin_9), U12.11 (O4)
- new net ~{0xA0}: J4.11 (Pin_11), U12.10 (O5)
- new net ~{0xCO}: J4.13 (Pin_13), U12.9 (O6)
- new net ~{0xE0}: J4.15 (Pin_15), U12.7 (O7)
- new net ~{MEG0_LO}: U15.22 (CE#), U2.11
- new net ~{MEG0}: TP1.1, U1.1, U2.12, U2.8
- no-connect marks 9 -> 15
Other:
- note removed: "BANK ZERO"
- note removed: "BUFFER_CLK +10ns"
- note removed: "BUS ENABLE"
- note removed: "CLK"
- note removed: "CLOCK PHASES"
- note removed: "CPU & BUS MANAGEMENT"
- note removed: "Generates a ~{RST} pulse of 150ms + 3 clock rising edges Ensures the CPU registers the reset even with slow or stopped clock"
- note removed: "I/O CONTROL"
- note removed: "M/X DEMUX"
- note removed: "Note: 74'112 triggers on the falling edge of the clock, whereas 74'74 triggers on the rising edge"
- note removed: "READY PIN"
- note removed: "READ_CLK +10ns (falling-edge only)"
- note removed: "RESET"
- note removed: "SYNC"
- note removed: "Two delay lines options: DS1035M-10 is DIP but obsolete DS1135Z-10 is a drop-in SMD replacement that is still active"
- note removed: "WRITE_CLK -20ns"
- note removed: "pull-down on buffer data bus is useful if you stop the clock, since the data bus is only driven for half the cycle pull-up/down on address bus and cpu data bus are useful only if you plan to tie BE low with nothing else driving the bus"
- note removed: "~{MR} is open-collector Do not connect to logic gate output directly"
- moved on the sheet: C1, C2, C3, C4, D1, H1, H2, J1, R11, R12, R6, TP1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

Commit message: Before PCB update
Parts:
- removed TP1: ~{MEG0}, TestPoint:TestPoint_THTPad_D1.5mm_Drill0.7mm, symbol Connector:TestPoint
- removed TP2: ~{MEG0_LO}, TestPoint:TestPoint_THTPad_D1.5mm_Drill0.7mm, symbol Connector:TestPoint
- removed TP3: MEG0_HI, TestPoint:TestPoint_THTPad_D1.5mm_Drill0.7mm, symbol Connector:TestPoint
- removed TP4: ~{BANK0_HI}, TestPoint:TestPoint_THTPad_D1.5mm_Drill0.7mm, symbol Connector:TestPoint
- removed TP5: ~{BANK0_LO}, TestPoint:TestPoint_THTPad_D1.5mm_Drill0.7mm, symbol Connector:TestPoint
- removed TP6: ~{ROM_OE}, TestPoint:TestPoint_THTPad_D1.5mm_Drill0.7mm, symbol Connector:TestPoint
- removed TP7: ~{PAGE1}, TestPoint:TestPoint_THTPad_D1.5mm_Drill0.7mm, symbol Connector:TestPoint
- added J5: Decoder Output, Connector_PinHeader_2.54mm:PinHeader_2x16_P2.54mm_Vertical, symbol Connector_Generic:Conn_02x08_Odd_Even
- C10, C11, C12, C13, C14, C15, C5, C6, C7, C8, C9: symbol Device:C -> Device:C_Small
Connections:
- net GND: now also U9.1 (~{R}), U9.2 (D), U9.3 (C), J5.10 (Pin_10), J5.12 (Pin_12), J5.14 (Pin_14), J5.15 (Pin_15), J5.16 (Pin_16), J5.2 (Pin_2), J5.4 (Pin_4), J5.6 (Pin_6), J5.8 (Pin_8)
- net MEG0_HI: now also J5.5 (Pin_5)
- net VCC: now also U9.4 (~{S})
- net ~{BANK0_HI}: now also J5.7 (Pin_7)
- net ~{BANK0_LO}: now also J5.9 (Pin_9)
- net ~{MEG0_LO}: now also J5.3 (Pin_3)
- net ~{MEG0}: now also J5.1 (Pin_1)
- net ~{PAGE1}: now also J5.13 (Pin_13)
- net ~{ROM_OE}: now also J5.11 (Pin_11)
- no-connect marks 15 -> 17
Other:
- note added: "Decoder Output"
- note removed: "TEST POINTS"
- moved on the sheet: C10, C11, C12, C13, C14, C15, C2, C4, C5, C6, C7, C8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

Commit message: More preening.
Parts:
- J4: value Conn_02x8_Odd_Even -> I/O
Connections:
- net GND: now also U12.4 (E1), U12.8 (GND)
Other:
- note added: "* ROM mapped in upper half of Bank 0 $8000-$FFFF * Page 1 is decoded into 8 slots for I/O * In Emulation mode, ROM is read. In Native mode, RAM is read. * Writes to RAM always take place even when read-shadowed by ROM. * Writes to ROM may take place in Emulation mode. * Two crystals provided, one for Emulation (ROM is slow), one for Native. * Module signals when upper half of first megabyte is ad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"
- note added: "BB816 512 KB Memory Module"
- moved on the sheet: C1, C3, D1, J1, R6

Commit message: New pcb
Parts:
- removed R11: 3.3k, Resistor_THT:R_Axial_DIN0207_L6.3mm_D2.5mm_P7.62mm_Horizontal, symbol Device:R_Small
- removed R12: 100k, Resistor_THT:R_Axial_DIN0207_L6.3mm_D2.5mm_P7.62mm_Horizontal, symbol Device:R_Small
- removed unit 5 of U4
- removed U5: 74LS32, Package_DIP:DIP-14_W7.62mm, symbol 74xx:74LS32
- removed U7: 74AHC125, Package_DIP:DIP-14_W7.62mm, symbol 74xx:74LS125
- removed U9: 74HC74, Package_DIP:DIP-14_W7.62mm, symbol 74xx:74LS74
- removed X1: 8MHz, Oscillator:Oscillator_DIP-8, symbol Oscillator:CXO_DIP8
- removed X2: 16MHz, Oscillator:Oscillator_DIP-8, symbol Oscillator:CXO_DIP8
- added J7: VP_REWR, Connector_PinHeader_2.54mm:PinHeader_2x05_P2.54mm_Vertical, symbol Connector_Generic:Conn_02x05_Odd_Even
- added unit 5 of U5
- added unit 4 of U5
- added unit 3 of U5
- C10, C11, C12, C13, C14, C15, C5, C6, C7, C8, C9: footprint (none) -> Capacitor_THT:C_Disc_D3.4mm_W2.1mm_P2.50mm
- J4, J5: footprint Connector_PinHeader_2.54mm:PinHeader_2x16_P2.54mm_Vertical -> Connector_PinHeader_2.54mm:PinHeader_2x08_P2.54mm_Vertical
- renumbered U10 to U5, U4 to U5
Connections:
- net A1: now also J7.10 (Pin_10); no longer J3.17 (Pin_17)
- net A2: now also J7.8 (Pin_8); no longer J3.15 (Pin_15)
- net A3: now also J7.6 (Pin_6); no longer J3.13 (Pin_13)
- net A4: now also J7.4 (Pin_4); no longer J3.11 (Pin_11)
- net E: now also U5.5; no longer U1.13, U5.2
- net GND: now also U1.13, U6.8 (GND), U8.8 (GND), J7.2 (Pin_2), U5.7 (GND)
- net VCC: now also U5.14 (VCC)
- net ~{VP}: now also J7.1 (Pin_1)
- net at U1.8: now also U5.4; no longer U5.1
- net at U3.12: now also U5.6; no longer U5.3
- new net: U5.10, U5.12, U5.13, U5.9
- new net AA1: J3.17 (Pin_17), J7.9 (Pin_9)
- new net AA2: J3.15 (Pin_15), J7.7 (Pin_7)
- new net AA3: J3.13 (Pin_13), J7.5 (Pin_5)
- new net AA4: J3.11 (Pin_11), J7.3 (Pin_3)
- no-connect marks 17 -> 19
Other:
- added sheet Vector Pull Rewrite (vpr.kicad_sch)
- note removed: "CLOCK"
- moved on the sheet: J2, J3, J4, U12, U14, U15, U1A, U1B, U1C, U1D, U1E, U1F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
