File: kohlbecker/BB816/hardware/AronnaxMemory/AronnaxMemory.kicad_pcb (KiCad board)
At the start: 4 copper layers, 152.4 x 64.8 mm, 29 parts, among them J1 Barrel_Jack_Switch, J2 Conn_02x40_Odd_Even, J3 Conn_02x18_Odd_Even, J5 I/O ~{CS}, J9 Vector Rewrite, U1 74LS04, U10 74HC30, U12 AS6C4008-55PCN, U13 AT28C256-15PC, U3 74LS32, U4 74LS08, U6 74LS32, U9 CD4072B

Commit message: ATF22V10
Parts:
- removed J9: Vector Rewrite, Connector_PinHeader_2.54mm:PinHeader_2x11_P2.54mm_Vertical
- removed U1: 74LS04, Package_DIP:DIP-14_W7.62mm
- removed U10: 74HC30, Package_DIP:DIP-14_W7.62mm
- removed U12: AS6C4008-55PCN, Package_DIP:DIP-32_W15.24mm
- removed U4: 74LS08, Package_DIP:DIP-14_W7.62mm
- removed U6: 74LS32, Package_DIP:DIP-14_W7.62mm
- removed U9: CD4072B, Package_DIP:DIP-14_W7.62mm
- added J6: 2M Sel, Connector_PinHeader_2.54mm:PinHeader_2x10_P2.54mm_Vertical, F.Cu at (87.1, 67.5)
- added U2: ATF22V10, Package_DIP:DIP-24_W7.62mm_Socket, F.Cu at (64.0, 81.3)
- added U5: ATF22V10, Package_DIP:DIP-24_W7.62mm_Socket, F.Cu at (109.2, 118.6)
- U13: footprint Socket:DIP_Socket-28_W11.9_W12.7_W15.24_W17.78_W18.5_3M_228-1277-00-0602J -> Package_DIP:DIP-28_W15.24mm_Socket
- U3: value 74LS32 -> ATF22V10; footprint Package_DIP:DIP-14_W7.62mm -> Package_DIP:DIP-24_W7.62mm_Socket
- moved C5 142.2 mm to (1.07, 1.32), turned to 0 degrees
- moved C9 91.9 mm to (183.0, 103.7)
- moved C7 90.8 mm to (183.0, 100.0), turned to 0 degrees
- moved C2 76.9 mm to (183.0, 92.8), turned to 0 degrees
- moved U3 71.2 mm to (47.7, 94.0), turned to 90 degrees
- moved C1 70.2 mm to (183.0, 89.1), turned to 0 degrees
- moved C11 70.0 mm to (183.0, 111.0)
- moved C3 67.1 mm to (183.0, 96.4), turned to 0 degrees
- moved C10 64.2 mm to (183.0, 107.3), turned to 0 degrees
- moved J5 17.9 mm to (59.1, 67.5)
- moved U13 16.7 mm to (133.5, 92.1)
- moved C4 13.9 mm to (133.4, 73.8), turned to 0 degrees
Connections:
- net ~{WR} renamed /~{WR}
- J2 pad 37: /~{RD} -> ~{RD}
- J5 pad 10: unconnected-(J5-Pin_10-Pad10) -> ~{IRQ5}
- J5 pad 12: unconnected-(J5-Pin_12-Pad12) -> ~{IO_5}
- J5 pad 14: unconnected-(J5-Pin_14-Pad14) -> ~{IRQ4}
- J5 pad 16: unconnected-(J5-Pin_16-Pad16) -> ~{IO_4}
- J5 pad 18: unconnected-(J5-Pin_18-Pad18) -> ~{IRQ3}
- J5 pad 2: ~{MEG0_HI} -> ~{IRQ7}
- J5 pad 20: unconnected-(J5-Pin_20-Pad20) -> ~{IO_3}
- J5 pad 4: ~{PAGE1} -> ~{IO_7}
- J5 pad 6: unconnected-(J5-Pin_6-Pad6) -> ~{IRQ6}
- J5 pad 8: unconnected-(J5-Pin_8-Pad8) -> ~{IO_6}
- U13 pad 6: /A4 -> /AA4
- U13 pad 7: /A3 -> /AA3
- U13 pad 8: /A2 -> /AA2
- U13 pad 9: /A1 -> /AA1
- U3 pad 1: /~{A15} -> unconnected-(U3-CLK-Pad1)
- U3 pad 10: PAGE1 -> ~{I/O}
- U3 pad 11: /~{BANK0_LO} -> unconnected-(U3-I-Pad11)
- U3 pad 12: /~{BANK0} -> unconnected-(U3-GND-Pad12)
- U3 pad 13: /A15 -> unconnected-(U3-I-Pad13)
- U3 pad 14: VCC -> unconnected-(U3-O-Pad14)
- U3 pad 2: /~{BANK0} -> /A7
- U3 pad 3: ~{BANK0_HI} -> /A6
- U3 pad 4: Net-(U1-Pad10) -> /A5
- U3 pad 5: ~{BANK0_HI} -> /A4
- U3 pad 6: ~{ROM_OE} -> /A3
- U3 pad 7: GND -> /A2
- U3 pad 8: ~{MEG0_LO_OE} -> /A1
- U3 pad 9: Net-(U3-Pad9) -> /A0
Routing:
- net /~{WR}: track 134.9 -> 0.00 mm
- net /E: track 127.1 -> 0.00 mm
- net /A15: track 110.9 -> 0.00 mm, vias 1 -> 0
- net /A10: track 103.7 -> 0.00 mm
- net /A11: track 93.7 -> 0.00 mm
- net /A9: track 86.3 -> 0.00 mm
- net /A13: track 84.0 -> 0.00 mm
- net /A8: track 81.8 -> 0.00 mm
- net /A12: track 81.1 -> 0.00 mm
- net /~{BANK0}: track 80.9 -> 0.00 mm, vias 2 -> 0
- net /A17: track 70.0 -> 0.00 mm, vias 1 -> 0
- net /A19: track 68.3 -> 0.00 mm
- net ~{BANK0_HI}: track 67.5 -> 0.00 mm
- net ~{MEG0_LO}: track 66.5 -> 0.00 mm
- net /D4: track 59.3 -> 0.00 mm
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
Commit message: PLAs for Days! Also Vector Rewrite
Parts:
- added D2: 1N4148, Diode_THT:D_DO-35_SOD27_P7.62mm_Horizontal, F.Cu at (115.9, 106.8)
- added D3: 1N4148, Diode_THT:D_DO-35_SOD27_P7.62mm_Horizontal, F.Cu at (119.4, 106.8)
- added RN1: 100k, Resistor_THT:R_Array_SIP9, F.Cu at (89.9, 106.2)
- added U4: 74HC283, Package_DIP:DIP-16_W7.62mm_Socket, F.Cu at (94.2, 106.3)
- added U89: 74LS348, Package_DIP:DIP-16_W7.62mm_Socket, F.Cu at (94.2, 94.6)
- moved J5 9.23 mm to (50.8, 63.5)
- moved U2 9.01 mm to (55.9, 77.5)
- moved J6 9.01 mm to (79.0, 63.6)
Connections:
- J2 pad 49: /~{VP} -> ~{VP}
- U3 pad 11: unconnected-(U3-I-Pad11) -> ~{VP}
- U3 pad 14: unconnected-(U3-O-Pad14) -> ~{VP_REWRITE}
Other:
- board size 152.4 x 64.8 mm -> 152.4 x 69.8 mm

Commit message: Heal board
Parts:
- removed J5: I/O ~{CS}, Connector_PinHeader_2.54mm:PinHeader_2x10_P2.54mm_Vertical
- removed J6: 2M Sel, Connector_PinHeader_2.54mm:PinHeader_2x10_P2.54mm_Vertical
- added J4: I/O, Connector_PinHeader_2.54mm:PinHeader_2x18_P2.54mm_Vertical, F.Cu at (132.1, 53.3)
- added J8: RAM, Connector_PinHeader_2.54mm:PinHeader_2x40_P2.54mm_Vertical, F.Cu at (27.9, 53.3)
Connections:
- net /~{WR} renamed ~{WR}
- U2 pad 23: unconnected-(U2-O-Pad23) -> ~{RAM_RD}
Other:
- board size 152.4 x 69.8 mm -> 152.4 x 64.8 mm

Commit message: Everything, except the plot.
Parts:
- removed C11: 100nF, Capacitor_THT:C_Disc_D3.4mm_W2.1mm_P2.50mm
- removed C12: 220u, Capacitor_THT:CP_Radial_D6.3mm_P2.50mm
- removed C13: 10u, Capacitor_THT:CP_Radial_D4.0mm_P1.50mm
- removed RN1: 100k, Resistor_THT:R_Array_SIP9
- removed U13: AT28C256-15PC, Package_DIP:DIP-28_W15.24mm_Socket
- removed U89: 74LS348, Package_DIP:DIP-16_W7.62mm_Socket
- added C21: 220u, Capacitor_THT:CP_Radial_D6.3mm_P2.50mm, F.Cu at (39.5, 90.8)
- added C22: 10u, Capacitor_THT:CP_Radial_D4.0mm_P1.50mm, F.Cu at (38.3, 96.9)
- added C6: 100nF, Capacitor_THT:C_Disc_D3.4mm_W2.1mm_P2.50mm, F.Cu at (46.5, 73.7)
- added C8: 100nF, Capacitor_THT:C_Disc_D3.4mm_W2.1mm_P2.50mm, F.Cu at (153.4, 75.7)
- added J9: RAM1, Connector_PinHeader_2.54mm:PinHeader_2x25_P2.54mm_Vertical, F.Cu at (39.2, 70.4)
- added R11: 3.3k, Resistor_THT:R_Axial_DIN0207_L6.3mm_D2.5mm_P7.62mm_Horizontal, F.Cu at (65.0, 120.8)
- added R12: 100k, Resistor_THT:R_Axial_DIN0207_L6.3mm_D2.5mm_P7.62mm_Horizontal, F.Cu at (69.1, 120.8)
- added RN2: 100k, Resistor_THT:R_Array_SIP9, F.Cu at (168.0, 106.7)
- added U10: ATF22V10, Package_DIP:DIP-24_W7.62mm_Socket, F.Cu at (75.9, 121.4)
- added U6: AS6C4008-55PCN, Package_DIP:DIP-32_W15.24mm_Socket, F.Cu at (46.5, 91.8)
- added U7: AT28C256-15PC, Socket:DIP_Socket-28_W11.9_W12.7_W15.24_W17.78_W18.5_3M_228-1277-00-0602J, F.Cu at (98.9, 95.1)
- added U8: ATF22V10, Package_DIP:DIP-24_W7.62mm_Socket, F.Cu at (142.9, 75.7)
- added U9: ATF22V10, Package_DIP:DIP-24_W7.62mm_Socket, F.Cu at (107.8, 121.0)
- added X1: 28MHz, Oscillator:Oscillator_DIP-8, F.Cu at (29.0, 116.0)
- J8: value RAM -> RAM0; footprint Connector_PinHeader_2.54mm:PinHeader_2x40_P2.54mm_Vertical -> Connector_PinHeader_2.54mm:PinHeader_2x25_P2.54mm_Vertical
- U2: value ATF22V10 -> 74HC74; footprint Package_DIP:DIP-24_W7.62mm_Socket -> Package_DIP:DIP-14_W7.62mm
- U3: value ATF22V10 -> 74AHC125; footprint Package_DIP:DIP-24_W7.62mm_Socket -> Package_DIP:DIP-14_W7.62mm
- U4: value 74HC283 -> ATF22V10; footprint Package_DIP:DIP-16_W7.62mm_Socket -> Package_DIP:DIP-24_W7.62mm_Socket
- U5: value ATF22V10 -> 74LS348; footprint Package_DIP:DIP-24_W7.62mm_Socket -> Package_DIP:DIP-16_W7.62mm_Socket
- moved C5 181.8 mm to (164.1, 81.8), turned to -90 degrees
- moved C1 154.8 mm to (29.0, 104.1)
- moved C3 140.4 mm to (43.1, 108.6)
- moved C2 139.7 mm to (43.3, 95.5)
- moved C10 107.1 mm to (76.0, 110.9)
- moved C7 88.2 mm to (98.8, 73.9)
- moved D3 80.5 mm to (169.4, 43.7), turned to 180 degrees
- moved J8 78.8 mm to (104.9, 70.4)
- moved D2 77.5 mm to (170.7, 51.9), turned to 180 degrees
- moved C9 75.6 mm to (107.7, 111.0)
- moved U5 57.7 mm to (153.5, 81.8), turned to 0 degrees
- moved U4 48.2 mm to (139.9, 121.5)
- moved J4 48.1 mm to (172.7, 79.0), turned to 0 degrees
- moved C4 37.7 mm to (140.0, 111.0)
- moved U2 30.9 mm to (43.3, 105.7)
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Connections:
- D2 pad 2: /~{NMI} -> unconnected-(D2-A-Pad2)
- D3 pad 1: VCC -> Net-(D3-K)
- D3 pad 2: /~{IRQ} -> ~{IRQ}
- J2 pad 11: /~{CLK_EN} -> ~{CLK_EN}
- J2 pad 19: /~{IRQ} -> ~{IRQ}
- J2 pad 41: /~{BANK0} -> ~{BANK0}
- J2 pad 43: /E -> E
- J2 pad 49: ~{VP} -> /~{VP}
- J4 pad 1: VCC -> ~{IO_0}
- J4 pad 10: GND -> VCC
- J4 pad 11: ~{IRQ5} -> ~{IRQ2}
- J4 pad 13: ~{IO_5} -> ~{IO_3}
- J4 pad 14: GND -> VCC
- J4 pad 15: ~{IRQ4} -> ~{IRQ3}
- J4 pad 18: GND -> VCC
- J4 pad 19: ~{IRQ3} -> ~{IRQ4}
- J4 pad 2: GND -> VCC
- J4 pad 21: ~{IO_3} -> ~{IO_5}
- J4 pad 22: GND -> VCC
- J4 pad 23: ~{IRQ2} -> ~{IRQ5}
- J4 pad 25: ~{IO_2} -> ~{IO_6}
- J4 pad 26: GND -> VCC
- J4 pad 27: ~{IRQ1} -> ~{IRQ6}
- J4 pad 29: ~{IO_1} -> ~{IO_7}
- J4 pad 3: ~{IRQ7} -> ~{IRQ0}
- J4 pad 30: GND -> VCC
- J4 pad 31: ~{IRQ0} -> ~{IRQ7}
- J4 pad 33: ~{IO_0} -> (no net)
- J4 pad 34: GND -> (no net)
- J4 pad 35: VCC -> (no net)
- J4 pad 36: GND -> (no net)
- J4 pad 5: ~{IO_7} -> ~{IO_1}
- J4 pad 6: GND -> VCC
- J4 pad 7: ~{IRQ6} -> ~{IRQ1}
- J4 pad 9: ~{IO_6} -> ~{IO_2}
- J8 pad 1: unconnected-(J8-Pin_1-Pad1) -> VCC
- J8 pad 10: Net-(J8-Pin_10) -> ~{WR}
- J8 pad 11: ~{MEGAB} -> /A20
- J8 pad 12: Net-(J8-Pin_10) -> /A19
- J8 pad 13: ~{MEG89} -> /A18
- J8 pad 14: Net-(J8-Pin_10) -> GND
- J8 pad 15: ~{MEG67} -> /A17
- J8 pad 16: Net-(J8-Pin_10) -> /A16
- J8 pad 17: ~{MEG45} -> /A15
- J8 pad 18: Net-(J8-Pin_10) -> /A14
- J8 pad 19: ~{MEG23} -> /A13
- J8 pad 2: Net-(J8-Pin_10) -> GND
- J8 pad 20: Net-(J8-Pin_10) -> VCC
- J8 pad 21: ~{MEG01} -> GND
- J8 pad 22: Net-(J8-Pin_10) -> /A12
- J8 pad 23: /A20 -> /A11
- J8 pad 24: Net-(J8-Pin_10) -> /A10
- J8 pad 25: /A19 -> /A9
- J8 pad 26: Net-(J8-Pin_10) -> /A8
- J8 pad 27: /A18 -> /A7
- J8 pad 28: Net-(J8-Pin_10) -> /A6
- J8 pad 29: /A17 -> /A5
- J8 pad 3: ~{WR} -> ~{MEG0}
- J8 pad 30: Net-(J8-Pin_10) -> GND
- J8 pad 31: /A16 -> /AA4
- J8 pad 32: Net-(J8-Pin_10) -> /AA3
- J8 pad 33: /A15 -> /AA2
- J8 pad 34: Net-(J8-Pin_10) -> /AA1
- J8 pad 35: /A14 -> /A0
- J8 pad 36: Net-(J8-Pin_10) -> VCC
- J8 pad 37: /A13 -> GND
- J8 pad 38: Net-(J8-Pin_10) -> /D7
- J8 pad 39: /A12 -> /D6
- J8 pad 4: Net-(J8-Pin_10) -> VCC
- J8 pad 40: Net-(J8-Pin_10) -> /D5
- J8 pad 41: /A11 -> /D4
- J8 pad 42: Net-(J8-Pin_10) -> /D3
- J8 pad 43: /A10 -> /D2
- J8 pad 44: Net-(J8-Pin_10) -> /D1
- J8 pad 45: /A9 -> /D0
- J8 pad 46: Net-(J8-Pin_10) -> GND
- J8 pad 47: /A8 -> (no net)
- J8 pad 48: Net-(J8-Pin_10) -> (no net)
- J8 pad 49: /A7 -> (no net)
- J8 pad 5: ~{RAM_OE} -> ~{MEG2}
- J8 pad 50: Net-(J8-Pin_10) -> (no net)
- J8 pad 6: Net-(J8-Pin_10) -> ~{MEG4}
- J8 pad 7: ~{MEGEF} -> GND
- J8 pad 8: Net-(J8-Pin_10) -> ~{MEG6}
- J8 pad 9: ~{MEGCD} -> ~{RAM_OE}
- U2 pad 1: ~{RD} -> unconnected-(U2A-~{R}-Pad1)
- U2 pad 10: ~{I/O} -> VCC
- U2 pad 11: ~{ROM_OE} -> /28MHz
- U2 pad 12: GND -> Net-(U2B-D)
- U2 pad 13: unconnected-(U2-I-Pad13) -> VCC
- U2 pad 14: unconnected-(U2-O-Pad14) -> VCC
- U2 pad 2: /A23 -> unconnected-(U2A-D-Pad2)
- U2 pad 3: /A22 -> unconnected-(U2A-C-Pad3)
- U2 pad 4: /A21 -> unconnected-(U2A-~{S}-Pad4)
- U2 pad 5: /A20 -> unconnected-(U2A-Q-Pad5)
- U2 pad 6: /A19 -> unconnected-(U2A-~{Q}-Pad6)
- U2 pad 7: /A18 -> GND
- U2 pad 8: /A17 -> Net-(U2B-D)
- U2 pad 9: /A16 -> /14MHz
- U3 pad 10: ~{I/O} -> E
- U3 pad 11: ~{VP} -> unconnected-(U3-Pad11)
- U3 pad 14: ~{VP_REWRITE} -> VCC
- U3 pad 2: /A7 -> unconnected-(U3-Pad2)
- U3 pad 3: /A6 -> unconnected-(U3-Pad3)
- U3 pad 4: /A5 -> unconnected-(U3-Pad4)
- U3 pad 5: /A4 -> unconnected-(U3-Pad5)
- U3 pad 6: /A3 -> unconnected-(U3-Pad6)
- U3 pad 7: /A2 -> GND
- U3 pad 8: /A1 -> /CLK_SRC
- U3 pad 9: /A0 -> /14MHz
- U4 pad 1: /AA3 -> unconnected-(U4-CLK-Pad1)
- U4 pad 10: /AA1 -> /~{VP}
- U4 pad 11: GND -> unconnected-(U4-I-Pad11)
- U4 pad 12: /A4 -> GND
- U4 pad 13: /AA2 -> unconnected-(U4-I-Pad13)
- U4 pad 14: /A3 -> unconnected-(U4-O-Pad14)
- U4 pad 15: /Y3 -> unconnected-(U4-O-Pad15)
- U4 pad 16: VCC -> ~{IRQ}
- U4 pad 2: /Y2 -> /A1
- U4 pad 4: /AA4 -> /A3
- U4 pad 5: /A1 -> /A4
- U4 pad 6: /Y1 -> E
- U4 pad 7: GND -> /Y1
- U4 pad 8: GND -> /Y2
- U4 pad 9: unconnected-(U4-C4-Pad9) -> /Y3
- U5 pad 1: unconnected-(U5-CLK-Pad1) -> ~{IRQ0}
- U5 pad 10: /A8 -> ~{IRQ7}
- U5 pad 11: /E -> ~{IRQ6}
- U5 pad 12: GND -> ~{IRQ5}
- U5 pad 13: unconnected-(U5-I-Pad13) -> ~{IRQ4}
- U5 pad 14: unconnected-(U5-O-Pad14) -> Net-(D3-K)
- U5 pad 15: unconnected-(U5-O-Pad15) -> ~{VP_REWRITE}
- U5 pad 16: unconnected-(U5-O-Pad16) -> VCC
- U5 pad 2: /~{BANK0} -> ~{IRQ1}
- U5 pad 3: /A15 -> ~{IRQ2}
- U5 pad 4: /A14 -> ~{IRQ3}
- U5 pad 5: /A13 -> GND
- U5 pad 6: /A12 -> /Y3
- U5 pad 7: /A11 -> /Y2
- U5 pad 8: /A10 -> GND
- U5 pad 9: /A9 -> /Y1
Routing:
- net ~{IRQ4}: track 0.00 -> 0.69 mm
Other:
- board text removed: "~{$80000}"
- board text removed: "~{0100}"
