File: kohlbecker/BB816/hardware/AronnaxMemory/AronnaxMemory.kicad_pcb (KiCad board)
At the start: 4 copper layers, 152.4 x 64.8 mm, 38 parts, among them J1 Barrel_Jack_Switch, J2 Conn_02x40_Odd_Even, J3 Conn_02x18_Odd_Even, J4 I/O, J8 RAM0, J9 RAM1, U10 ATF22V10, U2 74HC74, U3 74AHC125, U4 ATF22V10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

Commit message: Wow
Parts:
- removed D2: 1N4148, Diode_THT:D_DO-35_SOD27_P7.62mm_Horizontal
- removed RN2: 100k, Resistor_THT:R_Array_SIP9
- added R14: 10K, Resistor_THT:R_Axial_DIN0207_L6.3mm_D2.5mm_P7.62mm_Horizontal, F.Cu at (204.9, 113.7)
- added R3: 10K, Resistor_THT:R_Axial_DIN0207_L6.3mm_D2.5mm_P7.62mm_Horizontal, F.Cu at (191.8, 98.2)
- added R4: 10K, Resistor_THT:R_Axial_DIN0207_L6.3mm_D2.5mm_P7.62mm_Horizontal, F.Cu at (196.8, 113.7)
- added R5: 10K, Resistor_THT:R_Axial_DIN0207_L6.3mm_D2.5mm_P7.62mm_Horizontal, F.Cu at (200.8, 113.7)
- added RN1: 100k, Resistor_THT:R_Array_SIP9, F.Cu at (168.9, 103.5)
- moved D3 51.5 mm to (165.5, 95.0), turned to -90 degrees
- moved C8 6.48 mm to (146.9, 75.8)
- moved U8 6.48 mm to (136.4, 75.8)
- moved R6 5.93 mm to (28.8, 100.6), turned to 0 degrees
- moved C22 4.83 mm to (33.4, 96.8)
- moved C7 4.46 mm to (94.3, 73.5)
- moved U7 4.46 mm to (94.5, 94.7)
- moved C5 4.32 mm to (160.3, 83.8)
- moved U5 4.32 mm to (149.7, 83.8)
- moved C6 2.80 mm to (43.7, 73.8)
- moved U6 2.80 mm to (43.7, 91.9)
- moved C21 2.74 mm to (37.0, 91.8)
- moved C4 2.13 mm to (139.3, 109.0)
- moved U4 2.13 mm to (139.3, 119.5)
- moved C10 2.01 mm to (75.3, 109.0)
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Connections:
- net /Y1 renamed /ADDEND_AA1
- net /Y2 renamed /ADDEND_AA2
- net /Y3 renamed /ADDEND_AA3
- U5 pad 15: ~{VP_REWRITE} -> VCC
- U7 pad 22: unconnected-(U7-~{OE}-Pad22) -> ~{ROM_OE}

Commit message: New
Parts:
- J4: footprint Connector_PinHeader_2.54mm:PinHeader_2x18_P2.54mm_Vertical -> Connector_PinHeader_2.54mm:PinHeader_2x16_P2.54mm_Vertical
- J9: footprint Connector_PinHeader_2.54mm:PinHeader_2x25_P2.54mm_Vertical -> Connector_PinHeader_2.54mm:PinHeader_2x23_P2.54mm_Vertical

Commit message: Pare
Parts:
- added J5: I/O, Connector_PinHeader_2.54mm:PinHeader_2x24_P2.54mm_Vertical, F.Cu at (53.0, 70.5)
- added R13: 3.3k, Resistor_THT:R_Axial_DIN0207_L6.3mm_D2.5mm_P7.62mm_Horizontal, F.Cu at (51.0, 120.8)
- added R15: 100k, Resistor_THT:R_Axial_DIN0207_L6.3mm_D2.5mm_P7.62mm_Horizontal, F.Cu at (55.1, 120.8)
- added U1: W65C22SxP, Package_LCC:PLCC-44_THT-Socket, F.Cu at (69.8, 86.1)
- added U11: TL28L92IFR, footprints:FR44, F.Cu at (84.5, 80.1)
- added X2: 28MHz, Oscillator:Oscillator_DIP-8, F.Cu at (80.1, 102.0)
- J4: footprint Connector_PinHeader_2.54mm:PinHeader_2x16_P2.54mm_Vertical -> Connector_PinHeader_2.54mm:PinHeader_2x10_P2.54mm_Vertical
- J8: value RAM0 -> RAM CTL; footprint Connector_PinHeader_2.54mm:PinHeader_2x25_P2.54mm_Vertical -> Connector_PinHeader_2.54mm:PinHeader_2x09_P2.54mm_Vertical
- J9: value RAM1 -> IRQ A1-4; footprint Connector_PinHeader_2.54mm:PinHeader_2x23_P2.54mm_Vertical -> Connector_PinHeader_2.54mm:PinHeader_2x04_P2.54mm_Vertical
- U7: footprint Socket:DIP_Socket-28_W11.9_W12.7_W15.24_W17.78_W18.5_3M_228-1277-00-0602J -> Package_DIP:DIP-28_W15.24mm_Socket
- moved J9 111.0 mm to (150.2, 71.2)
- moved U6 69.4 mm to (106.2, 122.1)
- moved R14 59.6 mm to (158.5, 76.2), turned to 0 degrees
- moved U10 56.0 mm to (117.2, 82.3)
- moved C10 52.1 mm to (114.1, 74.2), turned to -90 degrees
- moved C2 46.5 mm to (51.9, 141.2)
- moved C9 35.7 mm to (71.8, 114.4), turned to -90 degrees
- moved R5 35.5 mm to (165.9, 107.4), turned to 180 degrees
- moved U9 32.6 mm to (74.7, 122.0)
- moved R4 32.3 mm to (165.9, 104.1), turned to 180 degrees
- moved R6 32.1 mm to (48.5, 75.2), turned to 90 degrees
- moved C22 29.5 mm to (43.7, 69.1)
- moved R3 26.0 mm to (165.9, 100.8), turned to 180 degrees
- moved U3 25.6 mm to (41.2, 93.1), turned to 0 degrees
- moved D1 22.3 mm to (42.9, 73.9), turned to 0 degrees
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Connections:
- net /28MHz renamed /TurboClock/28MHz
- J4 pad 1: ~{IO_0} -> ~{IO_3}
- J4 pad 11: ~{IRQ2} -> ~{IRQ5}
- J4 pad 13: ~{IO_3} -> ~{IO_6}
- J4 pad 15: ~{IRQ3} -> ~{IRQ6}
- J4 pad 17: ~{IO_4} -> ~{IO_7}
- J4 pad 19: ~{IRQ4} -> ~{IRQ7}
- J4 pad 3: ~{IRQ0} -> ~{IRQ3}
- J4 pad 5: ~{IO_1} -> ~{IO_4}
- J4 pad 7: ~{IRQ1} -> ~{IRQ4}
- J4 pad 9: ~{IO_2} -> ~{IO_5}
- J8 pad 1: VCC -> ~{MEGE}
- J8 pad 10: ~{WR} -> GND
- J8 pad 11: /A20 -> ~{MEG4}
- J8 pad 12: /A19 -> GND
- J8 pad 13: /A18 -> ~{MEG2}
- J8 pad 15: /A17 -> ~{MEG0}
- J8 pad 16: /A16 -> GND
- J8 pad 17: /A15 -> ~{RAM_OE}
- J8 pad 18: /A14 -> GND
- J8 pad 3: ~{MEG0} -> ~{MEGC}
- J8 pad 4: VCC -> GND
- J8 pad 5: ~{MEG2} -> ~{MEGA}
- J8 pad 6: ~{MEG4} -> GND
- J8 pad 7: GND -> ~{MEG8}
- J8 pad 8: ~{MEG6} -> GND
- J8 pad 9: ~{RAM_OE} -> ~{MEG6}
- J9 pad 1: VCC -> /AA4
- J9 pad 3: ~{MEGA} -> /AA3
- J9 pad 4: VCC -> GND
- J9 pad 5: ~{MEG8} -> /AA2
- J9 pad 6: ~{MEGC} -> GND
- J9 pad 7: GND -> /AA1
- J9 pad 8: ~{MEGE} -> GND
- R11 pad 1: E -> /TurboClock/E
- R12 pad 1: /CLK_SRC -> /TurboClock/CLK_SRC
- U10 pad 15: ~{MEGE} -> ~{MEG0}
- U10 pad 16: ~{MEGC} -> ~{MEG2}
- U10 pad 17: ~{MEGA} -> ~{MEG4}
- U10 pad 18: ~{MEG8} -> ~{MEG6}
- U10 pad 19: ~{MEG6} -> ~{MEG8}
- U10 pad 20: ~{MEG4} -> ~{MEGA}
- U10 pad 21: ~{MEG2} -> ~{MEGC}
- U10 pad 22: ~{MEG0} -> ~{MEGE}
- U2 pad 1: unconnected-(U2A-~{R}-Pad1) -> VCC
- U2 pad 2: unconnected-(U2A-D-Pad2) -> Net-(U2A-D)
- U2 pad 3: unconnected-(U2A-C-Pad3) -> /TurboClock/14MHz
- U2 pad 4: unconnected-(U2A-~{S}-Pad4) -> VCC
- U2 pad 5: unconnected-(U2A-Q-Pad5) -> /TurboClock/7MHz
- U2 pad 6: unconnected-(U2A-~{Q}-Pad6) -> Net-(U2A-D)
- U2 pad 9: /14MHz -> /TurboClock/14MHz
- U3 pad 1: unconnected-(U3-Pad1) -> /TurboClock/~E
- U3 pad 10: E -> /TurboClock/E
- U3 pad 2: unconnected-(U3-Pad2) -> /TurboClock/7MHz
- U3 pad 3: unconnected-(U3-Pad3) -> /TurboClock/CLK_SRC
- U3 pad 8: /CLK_SRC -> /TurboClock/CLK_SRC
- U3 pad 9: /14MHz -> /TurboClock/14MHz
- U4 pad 6: E -> unconnected-(U4-I-Pad6)
Routing:
- net ~{IRQ4}: track 0.69 -> 0.00 mm
Other:
- copper layers 4 -> 6
