File: kohlbecker/BB816/hardware/AronnaxMemory/AronnaxMemory.kicad_sch (KiCad schematic)
At the start: 29 parts, among them J1 Barrel_Jack_Switch, J2 Conn_02x40_Odd_Even, J3 Conn_02x18_Odd_Even, J5 I/O ~{CS}, J9 Vector Rewrite, U1 74LS04, U12 AS6C4008-55PCN, U13 AT28C256-15PC, U2 74LS32, U3 74LS32, U4 74LS08, U6 74LS32, U7 74LS32, U8 74LS138

Commit message: Saves
Connections:
- net ~{0x00}: now also J5.20 (Pin_20); no longer J5.2 (Pin_2)
- net ~{0x20}: now also J5.18 (Pin_18); no longer J5.4 (Pin_4)
- net ~{0x40}: now also J5.16 (Pin_16); no longer J5.6 (Pin_6)
- net ~{0x60}: now also J5.14 (Pin_14); no longer J5.8 (Pin_8)
- net ~{0x80}: now also J5.12 (Pin_12); no longer J5.10 (Pin_10)
- net ~{0xA0}: now also J5.10 (Pin_10); no longer J5.12 (Pin_12)
- net ~{0xCO}: now also J5.8 (Pin_8); no longer J5.14 (Pin_14)
- net ~{0xE0}: now also J5.6 (Pin_6); no longer J5.16 (Pin_16)
- net ~{MEG0_HI}: now also J5.2 (Pin_2); no longer J5.20 (Pin_20)
- net ~{PAGE1}: now also J5.4 (Pin_4); no longer J5.18 (Pin_18)
Other:
- moved on the sheet: J5
Changed lines of the file:
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@@
 	)
 	(junction
-		(at 389.89 254)
-		(diameter 0)
-		(color 0 0 0 0)
-	)
-	(junction
 		(at 58.42 105.41)
 		(diameter 0)
@@
 	)
 	(junction
+		(at 389.89 254)
+		(diameter 0)
+		(color 0 0 0 0)
+	)
+	(junction
 		(at 58.42 232.41)
 		(diameter 0)
@@
 		(exclude_from_sim no)
 		(in_bom yes)
-		(on_board yes)
+		(on_board no)
 		(dnp no)
 		(property "Reference" "J9"
@@
 	(symbol
 		(lib_id "Connector_Generic:Conn_02x10_Odd_Even")
-		(at 384.81 241.3 0)
-		(mirror y)
+		(at 384.81 243.84 180)
 		(unit 1)
 		(exclude_from_sim no)
@@
 		(dnp no)
 		(property "Reference" "J5"
-			(at 383.286 254 0)
+			(at 383.286 231.14 0)
 			(effects
 				(font
@@
 		)
 		(property "Value" "I/O ~{CS}"
-			(at 382.524 256.286 0)
+			(at 382.524 228.854 0)
 			(effects
 				(font
@@
 		)
 		(property "Footprint" "Connector_PinHeader_2.54mm:PinHeader_2x10_P2.54mm_Vertical"
-			(at 384.81 241.3 0)
+			(at 384.81 243.84 0)
 			(effects
 				(font
@@
 		)
 		(property "Datasheet" "~"
-			(at 384.81 241.3 0)
+			(at 384.81 243.84 0)
 			(effects
 				(font
@@
 		)
 		(property "Description" "Generic connector, double row, 02x10, odd/even pin numbering scheme (row 1 odd numbers, row 2 even numbers), script generated (kicad-library-utils/schlib/autogen/connector/)"
-			(at 384.81 241.3 0)
+			(at 384.81 243.84 0)
 			(effects
 				(font

Commit message: Memory
Connections:
- net ~{BANK0_HI}: now also U3.3, U3.5; no longer U3.2, U3.6
- net ~{BANK0}: now also U3.2; no longer U3.5
- net ~{ROM_OE}: now also U3.6; no longer U3.3
- net at U3.4: now also U1.2; no longer U1.6
- net at U3.1: now also U1.6; no longer U1.2
Other:
- added sheet VectorPullRewrite (VectorPullRewrite.kicad_sch)
- moved on the sheet: U3A, U3B
Changed lines of the file:
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@@
 	(symbol
 		(lib_id "74xx:74LS32")
-		(at 209.55 189.23 0)
+		(at 284.48 184.15 0)
 		(unit 2)
 		(exclude_from_sim no)
@@
 		(dnp no)
 		(property "Reference" "U3"
-			(at 209.804 188.976 0)
+			(at 284.734 183.896 0)
 			(effects
 				(font
@@
 		)
 		(property "Value" "74LS32"
-			(at 209.55 182.88 0)
+			(at 284.48 177.8 0)
 			(effects
 				(font
@@
 		)
 		(property "Footprint" "Package_DIP:DIP-14_W7.62mm"
-			(at 209.55 189.23 0)
+			(at 284.48 184.15 0)
 			(effects
 				(font
@@
 		)
 		(property "Datasheet" "http://www.ti.com/lit/gpn/sn74LS32"
-			(at 209.55 189.23 0)
+			(at 284.48 184.15 0)
 			(effects
 				(font
@@
 		)
 		(property "Description" "Quad 2-input OR"
-			(at 209.55 189.23 0)
+			(at 284.48 184.15 0)
 			(effects
 				(font
@@
 		(exclude_from_sim no)
 		(in_bom yes)
-		(on_board no)
+		(on_board yes)
 		(dnp no)
 		(property "Reference" "J9"
@@
 	(symbol
 		(lib_id "74xx:74LS32")
-		(at 284.48 184.15 0)
+		(at 209.55 189.23 0)
 		(unit 1)
 		(exclude_from_sim no)
@@
 		(dnp no)
 		(property "Reference" "U3"
-			(at 284.48 183.896 0)
+			(at 209.55 188.976 0)
 			(effects
 				(font
@@
 		)
 		(property "Value" "74LS32"
-			(at 284.48 177.8 0)
+			(at 209.55 182.88 0)
 			(effects
 				(font
@@
 		)
 		(property "Footprint" "Package_DIP:DIP-14_W7.62mm"
-			(at 284.48 184.15 0)
+			(at 209.55 189.23 0)
 			(effects
 				(font
@@
 		)
 		(property "Datasheet" "http://www.ti.com/lit/gpn/sn74LS32"
-			(at 284.48 184.15 0)
+			(at 209.55 189.23 0)
 			(effects
 				(font
@@
 		)
 		(property "Description" "Quad 2-input OR"
-			(at 284.48 184.15 0)
+			(at 209.55 189.23 0)
 			(effects
 				(font
@@
 				)
 			)
+		)
+	)
+	(sheet
+		(at 110.49 27.94)
+		(size 82.55 55.88)
+		(exclude_from_sim no)
+		(in_bom yes)
+		(on_board no)
+		(dnp no)
+		(fields_autoplaced yes)
+		(stroke
+			(width 0.1524)
+			(type solid)
+		)
+		(fill
+			(color 0 0 0 0.0000)
+		)
+		(property "Sheetname" "VectorPullRewrite"
+			(at 110.49 27.2284 0)
+			(effects
+				(font
+					(size 1.27 1.27)
+				)
+				(justify left bottom)
+			)
+		)
+		(property "Sheetfile" "VectorPullRewrite.kicad_sch"
+			(at 110.49 84.4046 0)
+			(effects
+				(font
+					(size 1.27 1.27)
+				)
+				(justify left top)
+			)
+		)
+		(instances
+			(project "AronnaxMemory"
+				(path "/f3290a4d-b1bc-4282-9c8a-cd936fe74ce9"
+					(page "2")
+				)
+			)

Commit message: Cleanup
Parts:
- removed C6, C8: 100nF, Capacitor_THT:C_Disc_D3.4mm_W2.1mm_P2.50mm, symbol Device:C
- removed unit 4 of U2
- removed unit 5 of U2
- removed unit 2 of U2
- removed unit 1 of U2
- removed unit 1 of U6
- removed U7: 74LS32, Package_DIP:DIP-14_W7.62mm, symbol 74xx:74LS32
- removed U8: 74LS138, Package_DIP:DIP-16_W7.62mm, symbol 74xx:74LS138
- added C10, C11: 100nF, Capacitor_THT:C_Disc_D3.4mm_W2.1mm_P2.50mm, symbol Device:C
- added U10: 74HC30, Package_DIP:DIP-14_W7.62mm, symbol BB816:74HC30
- added U9: CD4072B, Package_DIP:DIP-14_W7.62mm, symbol cd4072B:4072
- renumbered U2 to U6
Connections:
- net A10: now also U10.2; no longer U6.5
- net A11: now also U10.3
- net A12: now also U10.4
- net A13: now also U10.5
- net A14: now also U10.6
- net A15: now also U1.1, U3.13; no longer U1.5, U3.10
- net A19: now also U1.9, U6.2; no longer U1.11, U6.10
- net A20: now also U9.5
- net A21: now also U9.4
- net A22: now also U9.3
- net A23: now also U9.2
- net A8: now also U10.11
- net A9: now also U10.12; no longer U6.4
- net E: now also U1.11, U4.13; no longer U1.1, U4.5
- net GND: now also J9.15 (Pin_15), J9.17 (Pin_17), J9.19 (Pin_19), J9.21 (Pin_21), U1.5, U4.4, U4.5, U6.10, U6.4, U6.5, U6.9, C10.2, C11.2, U10.7 (GND), U9.10, U9.11, U9.12, U9.7 (VSS), U9.9; no longer U1.9, U4.12, U4.13
- net VCC: now also C10.1, C11.1, U10.14 (VCC), U9.14 (VDD)
- net ~{BANK0_HI}: now also U1.13; no longer U1.3
- net ~{BANK0_LO}: now also U3.11, U10.1; no longer U3.8
- net ~{BANK0}: now also U3.12; no longer U3.9
- net ~{MEG0_LO}: now also U6.3; no longer U6.8
- net ~{PAGE1}: now also U1.4; no longer U1.13
- net ~{ROM_OE}: no longer U13.22 (~{OE})
- net at U3.4: now also U1.10; no longer U1.2
- net at U6.6: no longer U6.9
- net ~{A19}: now reaches U1.8
- net ~{A19}: now also U6.12
- net at U4.11: now also U3.9
- net ~{MEG0}: now reaches U6.13
- net ~{MEG0}: now also U6.1, U9.1; no longer U6.9
- net ~{MEG0_LO_OE}: now reaches U12.24 (OE#)
- net ~{MEG0_LO_OE}: now also U3.8; no longer U3.11
- net at U4.6: no longer U3.12
- net at U1.12: now also U4.12; no longer U3.13
- net at U1.6: no longer U3.1
- net ~{0x00}: no longer names the net of J5.20 (Pin_20)
- net ~{0x20}: no longer names the net of J5.18 (Pin_18)
- net ~{0x40}: no longer names the net of J5.16 (Pin_16)
- net ~{0x60}: no longer names the net of J5.14 (Pin_14)
- net ~{0x80}: no longer names the net of J5.12 (Pin_12)
- net ~{0xA0}: no longer names the net of J5.10 (Pin_10)
- net ~{0xCO}: no longer names the net of J5.8 (Pin_8)
- net ~{0xE0}: no longer names the net of J5.6 (Pin_6)
- new net PAGE1: U1.3, U10.8, U3.10
- new net ~{A15}: U1.2, U3.1
- no-connect marks 5 -> 8
Other:
- removed sheet VectorPullRewrite
- moved on the sheet: C1, C12, C13, C2, C3, C4, C5, C7, C9, D1, H1, H2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

Commit message: ATF22V10
Parts:
- removed J9: Vector Rewrite, Connector_PinHeader_2.54mm:PinHeader_2x11_P2.54mm_Vertical, symbol Connector_Generic:Conn_02x11_Odd_Even
- removed U1: 74LS04, Package_DIP:DIP-14_W7.62mm, symbol 74xx:74LS04
- removed U10: 74HC30, Package_DIP:DIP-14_W7.62mm, symbol BB816:74HC30
- removed U12: AS6C4008-55PCN, Package_DIP:DIP-32_W15.24mm, symbol Memory_RAM:AS6C4008-55PCN
- removed U3, U6: 74LS32, Package_DIP:DIP-14_W7.62mm, symbol 74xx:74LS32
- removed U4: 74LS08, Package_DIP:DIP-14_W7.62mm, symbol 74xx:74LS08
- removed U9: CD4072B, Package_DIP:DIP-14_W7.62mm, symbol cd4072B:4072
- added J6: 2M Sel, Connector_PinHeader_2.54mm:PinHeader_2x10_P2.54mm_Vertical, symbol Connector_Generic:Conn_02x08_Odd_Even
- added U2, U3, U5: ATF22V10, Package_DIP:DIP-24_W7.62mm_Socket, symbol my:ATF22V10
- J5: symbol Connector_Generic:Conn_02x10_Odd_Even -> Connector_Generic:Conn_02x16_Odd_Even
- U13: footprint Socket:DIP_Socket-28_W11.9_W12.7_W15.24_W17.78_W18.5_3M_228-1277-00-0602J -> Package_DIP:DIP-28_W15.24mm_Socket
Connections:
- net A0: now also U3.9 (I)
- net A1: now also U3.8 (I); no longer U13.9 (A1)
- net A10: now also U5.8 (I)
- net A11: now also U5.7 (I)
- net A12: now also U5.6 (I)
- net A13: now also U5.5 (I)
- net A14: now also U5.4 (I)
- net A15: now also U5.3 (I)
- net A16: now also U2.9 (I)
- net A17: now also U2.8 (I)
- net A18: now also U2.7 (I)
- net A19: now also U2.6 (I)
- net A2: now also U3.7 (I); no longer U13.8 (A2)
- net A20: now also U2.5 (I)
- net A21: now also U2.4 (I)
- net A22: now also U2.3 (I)
- net A23: now also U2.2 (I)
- net A3: now also U3.6 (I); no longer U13.7 (A3)
- net A4: now also U3.5 (I); no longer U13.6 (A4)
- net A5: now also U3.4 (I)
- net A6: now also U3.3 (I)
- net A7: now also U3.2 (I)
- net A8: now also U5.10 (I)
- net A9: now also U5.9 (I)
- net AA1: now also U13.9 (A1)
- net AA2: now also U13.8 (A2)
- net AA3: now also U13.7 (A3)
- net AA4: now also U13.6 (A4)
- net E: now also U5.11 (I)
- net GND: now also J5.21 (Pin_21), J5.23 (Pin_23), J5.25 (Pin_25), J5.27 (Pin_27), J5.29 (Pin_29), J5.31 (Pin_31), J6.1 (Pin_1), J6.11 (Pin_11), J6.13 (Pin_13), J6.15 (Pin_15), J6.3 (Pin_3), J6.5 (Pin_5), J6.7 (Pin_7), J6.9 (Pin_9), U2.12 (GND), U5.12 (GND)
- net VCC: now also U2.24 (VCC), U5.24 (VCC)
- net ~{BANK0}: now also U5.2 (I)
- net ~{RD}: now also U2.1 (CLK)
- net ~{ROM_OE}: now also U2.11 (I), U5.22 (O)
- net ~{IRQ5}: now reaches J5.10 (Pin_10)
- net ~{IO_5}: now reaches J5.12 (Pin_12)
- net ~{IO_5}: now also U3.18 (O)
- net ~{IRQ4}: now reaches J5.14 (Pin_14)
- net ~{IO_4}: now reaches J5.16 (Pin_16)
- net ~{IO_4}: now also U3.19 (O)
- net ~{IRQ3}: now reaches J5.18 (Pin_18)
- net ~{IO_3}: now reaches J5.20 (Pin_20)
- net ~{IO_3}: now also U3.20 (O)
- net ~{IRQ6}: now reaches J5.6 (Pin_6)
- net ~{IO_6}: now reaches J5.8 (Pin_8)
- net ~{IO_6}: now also U3.17 (O)
- net ~{MEG0_HI} renamed ~{IRQ7}
- net ~{PAGE1} renamed ~{IO_7}
- net ~{IO_7}: now also U3.16 (O)
- new net ~{IO_0}: J5.32 (Pin_32), U3.23 (O)
- new net ~{IO_1}: J5.28 (Pin_28), U3.22 (O)
- new net ~{IO_2}: J5.24 (Pin_24), U3.21 (O)
- new net ~{IRQ0}: J5.30 (Pin_30)
- new net ~{IRQ1}: J5.26 (Pin_26)
- new net ~{IRQ2}: J5.22 (Pin_22)
- new net ~{I/O}: U2.10 (I), U3.10 (I), U5.23 (O)
- new net ~{MEG01}: J6.16 (Pin_16), U2.22 (O)
- new net ~{MEG23}: J6.14 (Pin_14), U2.21 (O)
- new net ~{MEG45}: J6.12 (Pin_12), U2.20 (O)
- new net ~{MEG67}: J6.10 (Pin_10), U2.19 (O)
- new net ~{MEG89}: J6.8 (Pin_8), U2.18 (O)
- new net ~{MEGAB}: J6.6 (Pin_6), U2.17 (O)
- new net ~{MEGCD}: J6.4 (Pin_4), U2.16 (O)
- new net ~{MEGEF}: J6.2 (Pin_2), U2.15 (O)
- new net ~{RAM_OE}: U5.21 (O)
- new net ~{STRETCH}: U5.20 (O)
- new net ~{TURBO}: U5.19 (O)
- no-connect marks 8 -> 1
Other:
- note added: "2 MB Segment Detection"
- note added: "32 KB ROM 0x008000-0x00FFFF"
- note added: "I/O CS"
- note added: "I/O CS+IRQ"
- note added: "I/O and ROM Area (Bank 0)"
- note added: "RAM always records. ROM is only enabled in Emulation"
- moved on the sheet: C12, C13, D1, J1, R6, U13

Commit message: PLAs for Days! Also Vector Rewrite
Parts:
- added D2, D3: 1N4148, Diode_THT:D_DO-35_SOD27_P7.62mm_Horizontal, symbol Diode:1N4148
- added J7: ~{IRQ7_NMI}, symbol Connector_Generic:Conn_02x02_Odd_Even
- added R1, R15: 1K, symbol Device:R
- added R13, R14, R3, R4, R5: 10K, symbol Device:R
- added RN1: 100k, Resistor_THT:R_Array_SIP9, symbol Device:R_Network08
- added U4: 74HC283, Package_DIP:DIP-16_W7.62mm_Socket, symbol Vega816:74HC283
- added U89: 74LS348, Package_DIP:DIP-16_W7.62mm_Socket, symbol 74xx:74LS348
Connections:
- net A1: now also U4.5 (A1)
- net A2: now also U4.3 (A2)
- net A3: now also U4.14 (A3)
- net A4: now also U4.12 (A4)
- net AA1: now also U4.10 (S4)
- net AA2: now also U4.13 (S3)
- net AA3: now also U4.1 (S2)
- net AA4: now also U4.4 (S1)
- net GND: now also R1.2, R15.2, R3.1, R4.1, R5.1, U4.11 (B4), U4.7 (C0), U4.8 (GND), U89.8 (GND)
- net VCC: now also D3.1 (K), J7.1 (Pin_1), R13.1, R14.1, U4.16 (VCC), U89.16 (VCC)
- net ~{IRQ0}: now also RN1.2 (R1), U89.4 (7)
- net ~{IRQ1}: now also RN1.3 (R2), U89.3 (6)
- net ~{IRQ2}: now also RN1.4 (R3), U89.2 (5)
- net ~{IRQ3}: now also RN1.5 (R4), U89.1 (4)
- net ~{IRQ4}: now also RN1.6 (R5), U89.13 (3)
- net ~{IRQ5}: now also RN1.7 (R6), U89.12 (2)
- net ~{IRQ6}: now also RN1.8 (R7), U89.11 (1)
- net ~{IRQ7}: now also J7.2 (Pin_2), J7.4 (Pin_4), RN1.9 (R8)
- net ~{IRQ}: now also D3.2 (A)
- net ~{NMI}: now also D2.2 (A)
- net ~{VP}: now also U3.11 (I)
- net ~{VP_REWRITE}: now reaches U3.14 (O)
- net ~{VP_REWRITE}: now also U89.5 (EI)
- new net: J7.3 (Pin_3), U89.10 (0)
- new net: R14.2, U89.14 (GS)
- new net: D2.1 (K), R13.2
- new net Y1: R5.2, U4.6 (B1), U89.9 (A0)
- new net Y2: R4.2, U4.2 (B2), U89.7 (A1)
- new net Y3: R3.2, U4.15 (B3), U89.6 (A2)
- no-connect marks 1 -> 3
Other:
- note added: "IRQ Priority"
- note added: "Reversed? Swap pins in symbol?"
- note added: "Vector Address Rewrite"
- note added: "~{VPB}+~{IRQ} Rewrite"
- note removed: "RAM always records. ROM is only enabled in Emulation"
- moved on the sheet: J2, J3, J5, J6, U13, U2, U3, U5

Commit message: Heal board
Parts:
- removed J5: I/O ~{CS}, Connector_PinHeader_2.54mm:PinHeader_2x10_P2.54mm_Vertical, symbol Connector_Generic:Conn_02x16_Odd_Even
- removed J6: 2M Sel, Connector_PinHeader_2.54mm:PinHeader_2x10_P2.54mm_Vertical, symbol Connector_Generic:Conn_02x08_Odd_Even
- added J4: I/O, Connector_PinHeader_2.54mm:PinHeader_2x18_P2.54mm_Vertical, symbol Connector_Generic:Conn_02x18_Odd_Even
- added J8: RAM, Connector_PinHeader_2.54mm:PinHeader_2x40_P2.54mm_Vertical, symbol Connector_Generic:Conn_02x40_Odd_Even
Connections:
- net A0: now also J8.63 (Pin_63)
- net A10: now also J8.43 (Pin_43)
- net A11: now also J8.41 (Pin_41)
- net A12: now also J8.39 (Pin_39)
- net A13: now also J8.37 (Pin_37)
- net A14: now also J8.35 (Pin_35)
- net A15: now also J8.33 (Pin_33)
- net A16: now also J8.31 (Pin_31)
- net A17: now also J8.29 (Pin_29)
- net A18: now also J8.27 (Pin_27)
- net A19: now also J8.25 (Pin_25)
- net A20: now also J8.23 (Pin_23)
- net A5: now also J8.53 (Pin_53)
- net A6: now also J8.51 (Pin_51)
- net A7: now also J8.49 (Pin_49)
- net A8: now also J8.47 (Pin_47)
- net A9: now also J8.45 (Pin_45)
- net AA1: now also J8.61 (Pin_61)
- net AA2: now also J8.59 (Pin_59)
- net AA3: now also J8.57 (Pin_57)
- net AA4: now also J8.55 (Pin_55)
- net D0: now also J8.79 (Pin_79)
- net D1: now also J8.77 (Pin_77)
- net D2: now also J8.75 (Pin_75)
- net D3: now also J8.73 (Pin_73)
- net D4: now also J8.71 (Pin_71)
- net D5: now also J8.69 (Pin_69)
- net D6: now also J8.67 (Pin_67)
- net D7: now also J8.65 (Pin_65)
- net GND: now also J4.10 (Pin_10), J4.12 (Pin_12), J4.14 (Pin_14), J4.16 (Pin_16), J4.18 (Pin_18), J4.2 (Pin_2), J4.20 (Pin_20), J4.22 (Pin_22), J4.24 (Pin_24), J4.26 (Pin_26), J4.28 (Pin_28), J4.30 (Pin_30), J4.32 (Pin_32), J4.34 (Pin_34), J4.36 (Pin_36), J4.4 (Pin_4), J4.6 (Pin_6), J4.8 (Pin_8)
- net VCC: now also J4.1 (Pin_1), J4.35 (Pin_35)
- net ~{IO_0}: now also J4.33 (Pin_33)
- net ~{IO_1}: now also J4.29 (Pin_29)
- net ~{IO_2}: now also J4.25 (Pin_25)
- net ~{IO_3}: now also J4.21 (Pin_21)
- net ~{IO_4}: now also J4.17 (Pin_17)
- net ~{IO_5}: now also J4.13 (Pin_13)
- net ~{IO_6}: now also J4.9 (Pin_9)
- net ~{IO_7}: now also J4.5 (Pin_5)
- net ~{IRQ0}: now also J4.31 (Pin_31)
- net ~{IRQ1}: now also J4.27 (Pin_27)
- net ~{IRQ2}: now also J4.23 (Pin_23)
- net ~{IRQ3}: now also J4.19 (Pin_19)
- net ~{IRQ4}: now also J4.15 (Pin_15)
- net ~{IRQ5}: now also J4.11 (Pin_11)
- net ~{IRQ6}: now also J4.7 (Pin_7)
- net ~{IRQ7}: now also J4.3 (Pin_3)
- net ~{MEG01}: now also J8.21 (Pin_21)
- net ~{MEG23}: now also J8.19 (Pin_19)
- net ~{MEG45}: now also J8.17 (Pin_17)
- net ~{MEG67}: now also J8.15 (Pin_15)
- net ~{MEG89}: now also J8.13 (Pin_13)
- net ~{MEGAB}: now also J8.11 (Pin_11)
- net ~{MEGCD}: now also J8.9 (Pin_9)
- net ~{MEGEF}: now also J8.7 (Pin_7)
- net ~{RAM_OE}: now also J8.5 (Pin_5)
- net ~{WR}: now also J8.3 (Pin_3)
- net ~{RAM_RD}: now reaches U2.23 (O)
- new net: J8.10 (Pin_10), J8.12 (Pin_12), J8.14 (Pin_14), J8.16 (Pin_16), J8.18 (Pin_18), J8.2 (Pin_2), J8.20 (Pin_20), J8.22 (Pin_22), J8.24 (Pin_24), J8.26 (Pin_26), J8.28 (Pin_28), J8.30 (Pin_30), J8.32 (Pin_32), J8.34 (Pin_34), J8.36 (Pin_36), J8.38 (Pin_38), J8.4 (Pin_4), J8.40 (Pin_40), J8.42 (Pin_42), J8.44 (Pin_44), J8.46 (Pin_46), J8.48 (Pin_48), J8.50 (Pin_50), J8.52 (Pin_52), J8.54 (Pin_54), J8.56 (Pin_56), J8.58 (Pin_58), J8.6 (Pin_6), J8.60 (Pin_60), J8.62 (Pin_62), J8.64 (Pin_64), J8.66 (Pin_66), J8.68 (Pin_68), J8.70 (Pin_70), J8.72 (Pin_72), J8.74 (Pin_74), J8.76 (Pin_76), J8.78 (Pin_78), J8.8 (Pin_8), J8.80 (Pin_80)
Other:
- note added: "I/O ~{CS}+~{IRQ}"
- note added: "RAM BUS"
- note removed: "I/O CS+IRQ"
- moved on the sheet: C1, C10, C11, C12, C13, C2, C3, C4, C5, C7, C9, D1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

Commit message: Everything, except the plot.
Parts:
- removed C11: 100nF, Capacitor_THT:C_Disc_D3.4mm_W2.1mm_P2.50mm, symbol Device:C
- removed J7: ~{IRQ7_NMI}, symbol Connector_Generic:Conn_02x02_Odd_Even
- removed R1, R15: 1K, symbol Device:R
- removed U4: 74HC283, Package_DIP:DIP-16_W7.62mm_Socket, symbol Vega816:74HC283
- added C6, C8: 100nF, Capacitor_THT:C_Disc_D3.4mm_W2.1mm_P2.50mm, symbol Device:C
- added J9: RAM1, Connector_PinHeader_2.54mm:PinHeader_2x25_P2.54mm_Vertical, symbol Connector_Generic:Conn_02x23_Odd_Even
- added R11: 3.3k, Resistor_THT:R_Axial_DIN0207_L6.3mm_D2.5mm_P7.62mm_Horizontal, symbol Device:R_Small
- added R12: 100k, Resistor_THT:R_Axial_DIN0207_L6.3mm_D2.5mm_P7.62mm_Horizontal, symbol Device:R_Small
- added U2: 74HC74, Package_DIP:DIP-14_W7.62mm, symbol 74xx:74LS74
- added U3: 74AHC125, Package_DIP:DIP-14_W7.62mm, symbol 74xx:74LS125
- added U4: ATF22V10, Package_DIP:DIP-24_W7.62mm_Socket, symbol my:ATF22V10
- added U6: AS6C4008-55PCN, Package_DIP:DIP-32_W15.24mm_Socket, symbol Memory_RAM:AS6C4008-55PCN
- added X1: 28MHz, Oscillator:Oscillator_DIP-8, symbol Oscillator:CXO_DIP8
- J4: symbol Connector_Generic:Conn_02x18_Odd_Even -> Connector_Generic:Conn_02x16_Odd_Even
- J8: value RAM -> RAM0; footprint Connector_PinHeader_2.54mm:PinHeader_2x40_P2.54mm_Vertical -> Connector_PinHeader_2.54mm:PinHeader_2x25_P2.54mm_Vertical; symbol Connector_Generic:Conn_02x40_Odd_Even -> Connector_Generic:Conn_02x23_Odd_Even
- R14, R3, R4, R5: footprint (none) -> Resistor_THT:R_Axial_DIN0207_L6.3mm_D2.5mm_P7.62mm_Horizontal
- U7: renamed from U13; footprint Package_DIP:DIP-28_W15.24mm_Socket -> Socket:DIP_Socket-28_W11.9_W12.7_W15.24_W17.78_W18.5_3M_228-1277-00-0602J
- renumbered C12 to C21, C13 to C22, U2 to U10, U89 to U5, U3 to U8, U5 to U9
Connections:
- net ~{STRETCH} is gone; now on net ~{CLK_EN}: U9.20 (O)
- net A0: now also J8.35 (Pin_35), U8.11 (I), J9.35 (Pin_35), U6.12 (A0); no longer J8.63 (Pin_63), U8.9 (I)
- net A1: now also U8.10 (I), J9.34 (Pin_34), U4.2 (I); no longer U8.8 (I)
- net A10: now also J8.24 (Pin_24), U8.1 (CLK), J9.24 (Pin_24), U6.23 (A10); no longer J8.43 (Pin_43)
- net A11: now also J8.23 (Pin_23), J9.23 (Pin_23), U6.25 (A11); no longer J8.41 (Pin_41)
- net A12: now also J8.22 (Pin_22), J9.22 (Pin_22), U6.4 (A12); no longer J8.39 (Pin_39)
- net A13: now also J8.19 (Pin_19), J9.19 (Pin_19), U6.28 (A13); no longer J8.37 (Pin_37)
- net A14: now also J8.18 (Pin_18), J9.18 (Pin_18), U6.3 (A14); no longer J8.35 (Pin_35)
- net A15: now also J8.17 (Pin_17), J9.17 (Pin_17), U6.31 (A15); no longer J8.33 (Pin_33)
- net A16: now also J8.16 (Pin_16), J9.16 (Pin_16), U6.2 (A16); no longer J8.31 (Pin_31)
- net A17: now also J8.15 (Pin_15), J9.15 (Pin_15), U6.30 (A17); no longer J8.29 (Pin_29)
- net A18: now also J8.13 (Pin_13), J9.13 (Pin_13), U6.1 (A18); no longer J8.27 (Pin_27)
- net A19: now also J8.12 (Pin_12), J9.12 (Pin_12); no longer J8.25 (Pin_25)
- net A2: now also U8.9 (I), J9.33 (Pin_33), U4.3 (I); no longer U8.7 (I)
- net A20: now also J8.11 (Pin_11), J9.11 (Pin_11); no longer J8.23 (Pin_23)
- net A3: now also U8.8 (I), J9.32 (Pin_32), U4.4 (I); no longer U8.6 (I)
- net A4: now also U8.7 (I), J9.31 (Pin_31), U4.5 (I); no longer U8.5 (I)
- net A5: now also J8.29 (Pin_29), U8.6 (I), J9.29 (Pin_29), U6.7 (A5); no longer J8.53 (Pin_53), U8.4 (I)
- net A6: now also J8.28 (Pin_28), U8.5 (I), J9.28 (Pin_28), U6.6 (A6); no longer J8.51 (Pin_51), U8.3 (I)
- net A7: now also J8.27 (Pin_27), U8.4 (I), J9.27 (Pin_27), U6.5 (A7); no longer J8.49 (Pin_49), U8.2 (I)
- net A8: now also J8.26 (Pin_26), U8.3 (I), J9.26 (Pin_26), U6.27 (A8); no longer J8.47 (Pin_47)
- net A9: now also J8.25 (Pin_25), U8.2 (I), J9.25 (Pin_25), U6.26 (A9); no longer J8.45 (Pin_45)
- net AA1: now also J8.34 (Pin_34), U4.17 (O), U6.11 (A1); no longer J8.61 (Pin_61)
- net AA2: now also J8.33 (Pin_33), U4.18 (O), U6.10 (A2); no longer J8.59 (Pin_59)
- net AA3: now also J8.32 (Pin_32), U4.19 (O), U6.9 (A3); no longer J8.57 (Pin_57)
- net AA4: now also J8.31 (Pin_31), U4.20 (O), U6.8 (A4); no longer J8.55 (Pin_55)
- net CLK_SRC: now also R12.1, U3.8
- net D0: now also J8.45 (Pin_45), J9.45 (Pin_45), U6.13 (DQ0); no longer J8.79 (Pin_79)
- net D1: now also J8.44 (Pin_44), J9.44 (Pin_44), U6.14 (DQ1); no longer J8.77 (Pin_77)
- net D2: now also J8.43 (Pin_43), J9.43 (Pin_43), U6.15 (DQ2); no longer J8.75 (Pin_75)
- net D3: now also J8.42 (Pin_42), J9.42 (Pin_42), U6.17 (DQ3); no longer J8.73 (Pin_73)
- net D4: now also J8.41 (Pin_41), J9.41 (Pin_41), U6.18 (DQ4); no longer J8.71 (Pin_71)
- net D5: now also J8.40 (Pin_40), J9.40 (Pin_40), U6.19 (DQ5); no longer J8.69 (Pin_69)
- net D6: now also J8.39 (Pin_39), J9.39 (Pin_39), U6.20 (DQ6); no longer J8.67 (Pin_67)
- net D7: now also J8.38 (Pin_38), J9.38 (Pin_38), U6.21 (DQ7); no longer J8.65 (Pin_65)
- net E: now also R11.1, U3.10, U4.6 (I)
- net GND: now also J8.14 (Pin_14), J8.2 (Pin_2), J8.21 (Pin_21), J8.30 (Pin_30), J8.37 (Pin_37), J8.46 (Pin_46), J8.7 (Pin_7), U5.5 (EI), U8.12 (GND), C6.2, C8.2, J9.14 (Pin_14), J9.2 (Pin_2), J9.21 (Pin_21), J9.30 (Pin_30), J9.37 (Pin_37), J9.46 (Pin_46), J9.7 (Pin_7), R11.2, R12.2, U2.7 (GND), U3.7 (GND), U4.12 (GND), U6.16 (VSS), X1.4 (GND); no longer J4.10 (Pin_10), J4.14 (Pin_14), J4.18 (Pin_18), J4.2 (Pin_2), J4.22 (Pin_22), J4.26 (Pin_26), J4.30 (Pin_30), J4.34 (Pin_34), J4.36 (Pin_36), J4.6 (Pin_6)
- net VCC: now also J4.10 (Pin_10), J4.14 (Pin_14), J4.18 (Pin_18), J4.2 (Pin_2), J4.22 (Pin_22), J4.26 (Pin_26), J4.30 (Pin_30), J4.6 (Pin_6), J8.1 (Pin_1), J8.20 (Pin_20), J8.36 (Pin_36), J8.4 (Pin_4), RN1.1 (common), U8.24 (VCC), C6.1, C8.1, J9.1 (Pin_1), J9.20 (Pin_20), J9.36 (Pin_36), J9.4 (Pin_4), U2.10 (~{S}), U2.13 (~{R}), U2.14 (VCC), U3.14 (VCC), U4.24 (VCC), U6.32 (VCC), X1.8 (Vcc); no longer D3.1 (K), J4.1 (Pin_1), J4.35 (Pin_35)
- net ~{IO_0}: now also J4.1 (Pin_1); no longer J4.33 (Pin_33)
- net ~{IO_1}: now also J4.5 (Pin_5); no longer J4.29 (Pin_29)
- net ~{IO_2}: now also J4.9 (Pin_9); no longer J4.25 (Pin_25)
- net ~{IO_3}: now also J4.13 (Pin_13); no longer J4.21 (Pin_21)
- net ~{IO_5}: now also J4.21 (Pin_21); no longer J4.13 (Pin_13)
- net ~{IO_6}: now also J4.25 (Pin_25); no longer J4.9 (Pin_9)
- net ~{IO_7}: now also J4.29 (Pin_29); no longer J4.5 (Pin_5)
- net ~{IRQ0}: now also J4.3 (Pin_3), RN1.9 (R8), U5.1 (4); no longer J4.31 (Pin_31), RN1.2 (R1), U5.4 (7)
- net ~{IRQ1}: now also J4.7 (Pin_7), RN1.8 (R7), U5.2 (5); no longer J4.27 (Pin_27), RN1.3 (R2), U5.3 (6)
- net ~{IRQ2}: now also J4.11 (Pin_11), RN1.7 (R6), U5.3 (6); no longer J4.23 (Pin_23), RN1.4 (R3), U5.2 (5)
- net ~{IRQ3}: now also J4.15 (Pin_15), RN1.6 (R5), U5.4 (7); no longer J4.19 (Pin_19), RN1.5 (R4), U5.1 (4)
- net ~{IRQ4}: now also J4.19 (Pin_19), RN1.5 (R4); no longer J4.15 (Pin_15), RN1.6 (R5)
- net ~{IRQ5}: now also J4.23 (Pin_23), RN1.4 (R3); no longer J4.11 (Pin_11), RN1.7 (R6)
- net ~{IRQ6}: now also J4.27 (Pin_27), RN1.3 (R2); no longer J4.7 (Pin_7), RN1.8 (R7)
- net ~{IRQ7}: now also J4.31 (Pin_31), RN1.2 (R1), U5.10 (0); no longer J4.3 (Pin_3), RN1.9 (R8)
- net ~{IRQ}: now also U4.16 (O)
- net ~{I/O}: now also U8.13 (I); no longer U8.10 (I)
- net ~{NMI}: now also U4.21 (O); no longer D2.2 (A)
- net ~{RAM_OE}: now also J8.9 (Pin_9), J9.9 (Pin_9); no longer J8.5 (Pin_5)
- net ~{VP_REWRITE}: now also U5.15 (E0); no longer U5.5 (EI), U8.14 (O)
- net ~{VP}: now also U4.10 (I); no longer U8.11 (I)
- net ~{WR}: now also J8.10 (Pin_10), J9.10 (Pin_10); no longer J8.3 (Pin_3)
- net at R14.2, U5.14 (GS): now also D3.1 (K)
- net Y1 renamed ADDEND_AA1
- net ADDEND_AA1: now also U4.7 (I)
- net Y2 renamed ADDEND_AA2
- net ADDEND_AA2: now also U4.8 (I)
- net Y3 renamed ADDEND_AA3
- net ADDEND_AA3: now also U4.9 (I)
- net ~{MEG01} renamed ~{MEG0}
- net ~{MEG0}: now also J8.3 (Pin_3); no longer J8.21 (Pin_21)
- net ~{MEG23} renamed ~{MEG2}
- net ~{MEG2}: now also J8.5 (Pin_5); no longer J8.19 (Pin_19)
- net ~{MEG45} renamed ~{MEG4}
- net ~{MEG4}: now also J8.6 (Pin_6); no longer J8.17 (Pin_17)
- net ~{MEG67} renamed ~{MEG6}
- net ~{MEG6}: now also J8.8 (Pin_8); no longer J8.15 (Pin_15)
- net ~{MEG89} renamed ~{MEG8}
- net ~{MEG8}: now also J9.5 (Pin_5); no longer J8.13 (Pin_13)
- net ~{MEGAB} renamed ~{MEGA}
- net ~{MEGA}: now also J9.3 (Pin_3); no longer J8.11 (Pin_11)
- net ~{MEGCD} renamed ~{MEGC}
- net ~{MEGC}: now also J9.6 (Pin_6); no longer J8.9 (Pin_9)
- net ~{MEGEF} renamed ~{MEGE}
- net ~{MEGE}: now also J9.8 (Pin_8); no longer J8.7 (Pin_7)
- net ~{TURBO}: no longer names the net of U9.19 (O)
- new net: U2.12 (D), U2.8 (~{Q})
- new net 14MHz: U2.9 (Q), U3.9
- new net 28MHz: U2.11 (C), X1.5 (OUT)
- no-connect marks 3 -> 2
Other:
- note added: "2MB Boundaries"
- note added: "32KB ROM 0x008000 0x00FFFF"
- note added: "512KB RAM 0x000000 0x07FFFF"
- note added: "A1-A4 Offset"
- note added: "Address Decode - IRQ Vector Pull Rewrite - Native Mode Turbo Clock - 512KB RAM - 32KB ROM"
- note added: "BB816 System Controller"
- note added: "Bank Address"
- note added: "Based on the BB816 Breakout Board by M. Adrien Kohlbecker"
- note added: "I/O Select"
- note added: "I/O+ROM Area"
- note added: "Memory 512KB RAM + 32KB ROM"
- note added: "Native Mode Only See 65816 datasheet section 2.28"
- note added: "Note: Not subject to ~{VP} Rewrite and associated delay. See 65816 datasheet 2.28"
- note added: "Note: ~{VP} Rewrite of A1-A4 applies only to low RAM bus. See 65816 datasheet 2.28"
- note added: "Power"
- note added: "Priority"
- note added: "RAM BUS 0 Low 8 MB"
- note added: "RAM BUS 1 High 8 MB"
- note added: "Turbo Clock"
- note added: "Vector Pull Rewrite"
- note added: "~{IRQ} Pullup"
- note removed: "2 MB Segment Detection"
- note removed: "32 KB ROM 0x008000-0x00FFFF"
- note removed: "I/O CS"
- note removed: "I/O and ROM Area (Bank 0)"
- note removed: "IRQ Priority"
- note removed: "POWER"
- note removed: "RAM BUS"
- note removed: "Vector Address Rewrite"
- note removed: "~{VPB}+~{IRQ} Rewrite"
- moved on the sheet: C1, C2, C21, C22, C3, C4, C5, D1, D2, D3, H1, H2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
