File: kohlbecker/BB816/hardware/AronnaxMemory/AronnaxMemory.kicad_sch (KiCad schematic)
At the start: 42 parts, among them J1 Barrel_Jack_Switch, J2 Conn_02x40_Odd_Even, J3 Conn_02x18_Odd_Even, J4 I/O, J8 RAM0, J9 RAM1, U10 ATF22V10, U2 74HC74, U3 74AHC125, U4 ATF22V10, U5 74LS348, U6 AS6C4008-55PCN, U7 AT28C256-15PC, U8 ATF22V10, U9 ATF22V10, X1 28MHz

Commit message: Wow
Parts:
- removed D2: 1N4148, Diode_THT:D_DO-35_SOD27_P7.62mm_Horizontal, symbol Diode:1N4148
- removed R13: 10K, symbol Device:R
Connections:
- net ~{VP_REWRITE} is gone; now on net VCC: U5.15 (E0)
- net ~{ROM_OE}: now also U7.22 (~{OE})
Other:
- note added: "Address Decode - IRQ Vector Pull Rewrite - Native Mode Turbo Clock - 512KB RAM - 32KB ROM CPLDs allow fine grain tuning. This design can implement the memory map of BigDumbMonkey's POC 1 design. This design implements section 2.28 of the 65816 datasheet. Shadow RAM allows banking out slower EEPROM once startup is complete."
- note added: "After M. Adrien Kohlbecker (BB816 Breakout v.A27)"
- note added: "BB816 Programmable System Controller"
- note added: "I/O Bus"
- note removed: "Address Decode - IRQ Vector Pull Rewrite - Native Mode Turbo Clock - 512KB RAM - 32KB ROM"
- note removed: "BB816 System Controller"
- note removed: "Based on the BB816 Breakout Board by M. Adrien Kohlbecker"
- note removed: "I/O ~{CS}+~{IRQ}"
- note removed: "~{IRQ} Pullup"
- moved on the sheet: C21, C22, D1, D3, J1, J2, J3, J4, J8, J9, R11, R12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
