File: kohlbecker/BB816/hardware/AronnaxMemory/AronnaxMemory.kicad_sch (KiCad schematic)
At the start: 40 parts, among them J1 Barrel_Jack_Switch, J2 Conn_02x40_Odd_Even, J3 Conn_02x18_Odd_Even, J4 I/O, J8 RAM0, J9 RAM1, U10 ATF22V10, U2 74HC74, U3 74AHC125, U4 ATF22V10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

Commit message: New
Parts:
- J4: footprint Connector_PinHeader_2.54mm:PinHeader_2x18_P2.54mm_Vertical -> Connector_PinHeader_2.54mm:PinHeader_2x16_P2.54mm_Vertical
- J9: footprint Connector_PinHeader_2.54mm:PinHeader_2x25_P2.54mm_Vertical -> Connector_PinHeader_2.54mm:PinHeader_2x23_P2.54mm_Vertical
Changed lines of the file:
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@@
 			)
 		)
-		(property "Footprint" "Connector_PinHeader_2.54mm:PinHeader_2x18_P2.54mm_Vertical"
+		(property "Footprint" "Connector_PinHeader_2.54mm:PinHeader_2x16_P2.54mm_Vertical"
 			(at 162.56 212.09 0)
 			(effects
@@
 			)
 		)
-		(property "Footprint" "Connector_PinHeader_2.54mm:PinHeader_2x25_P2.54mm_Vertical"
+		(property "Footprint" "Connector_PinHeader_2.54mm:PinHeader_2x23_P2.54mm_Vertical"
 			(at 379.73 213.36 0)
 			(effects

Commit message: Pare
Parts:
- removed J9: RAM1, Connector_PinHeader_2.54mm:PinHeader_2x23_P2.54mm_Vertical, symbol Connector_Generic:Conn_02x23_Odd_Even
- removed R11: 3.3k, Resistor_THT:R_Axial_DIN0207_L6.3mm_D2.5mm_P7.62mm_Horizontal, symbol Device:R_Small
- removed R12: 100k, Resistor_THT:R_Axial_DIN0207_L6.3mm_D2.5mm_P7.62mm_Horizontal, symbol Device:R_Small
- removed U2: 74HC74, Package_DIP:DIP-14_W7.62mm, symbol 74xx:74LS74
- removed U3: 74AHC125, Package_DIP:DIP-14_W7.62mm, symbol 74xx:74LS125
- removed X1: 28MHz, Oscillator:Oscillator_DIP-8, symbol Oscillator:CXO_DIP8
- added J5: I/O, Connector_PinHeader_2.54mm:PinHeader_2x24_P2.54mm_Vertical, symbol Connector_Generic:Conn_02x24_Odd_Even
- added J9: IRQ A1-4, Connector_PinHeader_2.54mm:PinHeader_2x04_P2.54mm_Vertical, symbol Connector_Generic:Conn_02x04_Odd_Even
- added U1: W65C22SxP, Package_LCC:PLCC-44_THT-Socket, symbol BB816:W65C22SxP
- added U11: TL28L92IFR, FR44, symbol TL28L92IFR:TL28L92IFR
- added X2: 28MHz, Oscillator:Oscillator_DIP-8, symbol Oscillator:CXO_DIP8
- J4: footprint Connector_PinHeader_2.54mm:PinHeader_2x16_P2.54mm_Vertical -> Connector_PinHeader_2.54mm:PinHeader_2x10_P2.54mm_Vertical; symbol Connector_Generic:Conn_02x16_Odd_Even -> Connector_Generic:Conn_02x10_Odd_Even
- J8: value RAM0 -> RAM CTL; footprint Connector_PinHeader_2.54mm:PinHeader_2x25_P2.54mm_Vertical -> Connector_PinHeader_2.54mm:PinHeader_2x09_P2.54mm_Vertical; symbol Connector_Generic:Conn_02x23_Odd_Even -> Connector_Generic:Conn_02x09_Odd_Even
- U7: footprint Socket:DIP_Socket-28_W11.9_W12.7_W15.24_W17.78_W18.5_3M_228-1277-00-0602J -> Package_DIP:DIP-28_W15.24mm_Socket
Connections:
- net A0: no longer J8.35 (Pin_35)
- net A10: no longer J8.24 (Pin_24)
- net A11: no longer J8.23 (Pin_23)
- net A12: no longer J8.22 (Pin_22)
- net A13: no longer J8.19 (Pin_19)
- net A14: no longer J8.18 (Pin_18)
- net A15: no longer J8.17 (Pin_17)
- net A16: no longer J8.16 (Pin_16)
- net A17: no longer J8.15 (Pin_15)
- net A18: no longer J8.13 (Pin_13)
- net A19: no longer J8.12 (Pin_12)
- net A20: no longer J8.11 (Pin_11)
- net A5: no longer J8.29 (Pin_29)
- net A6: no longer J8.28 (Pin_28)
- net A7: no longer J8.27 (Pin_27)
- net A8: no longer J8.26 (Pin_26)
- net A9: no longer J8.25 (Pin_25)
- net AA1: now also J9.7 (Pin_7); no longer J8.34 (Pin_34)
- net AA2: now also J9.5 (Pin_5); no longer J8.33 (Pin_33)
- net AA3: now also J9.3 (Pin_3); no longer J8.32 (Pin_32)
- net AA4: now also J9.1 (Pin_1); no longer J8.31 (Pin_31)
- net D0: no longer J8.45 (Pin_45)
- net D1: no longer J8.44 (Pin_44)
- net D2: no longer J8.43 (Pin_43)
- net D3: no longer J8.42 (Pin_42)
- net D4: no longer J8.41 (Pin_41)
- net D5: no longer J8.40 (Pin_40)
- net D6: no longer J8.39 (Pin_39)
- net D7: no longer J8.38 (Pin_38)
- net E: no longer U4.6 (I)
- net GND: now also J8.10 (Pin_10), J8.12 (Pin_12), J8.16 (Pin_16), J8.18 (Pin_18), J8.4 (Pin_4), J8.6 (Pin_6), J8.8 (Pin_8), J9.2 (Pin_2), J9.4 (Pin_4), J9.6 (Pin_6), J9.8 (Pin_8); no longer J4.24 (Pin_24), J4.28 (Pin_28), J4.32 (Pin_32), J8.21 (Pin_21), J8.30 (Pin_30), J8.37 (Pin_37), J8.46 (Pin_46), J8.7 (Pin_7)
- net VCC: no longer J4.22 (Pin_22), J4.26 (Pin_26), J4.30 (Pin_30), J8.1 (Pin_1), J8.20 (Pin_20), J8.36 (Pin_36), J8.4 (Pin_4)
- net ~{IO_0}: no longer J4.1 (Pin_1)
- net ~{IO_1}: no longer J4.5 (Pin_5)
- net ~{IO_2}: no longer J4.9 (Pin_9)
- net ~{IO_3}: now also J4.1 (Pin_1); no longer J4.13 (Pin_13)
- net ~{IO_4}: now also J4.5 (Pin_5); no longer J4.17 (Pin_17)
- net ~{IO_5}: now also J4.9 (Pin_9); no longer J4.21 (Pin_21)
- net ~{IO_6}: now also J4.13 (Pin_13); no longer J4.25 (Pin_25)
- net ~{IO_7}: now also J4.17 (Pin_17); no longer J4.29 (Pin_29)
- net ~{IRQ0}: no longer J4.3 (Pin_3)
- net ~{IRQ1}: no longer J4.7 (Pin_7)
- net ~{IRQ2}: no longer J4.11 (Pin_11)
- net ~{IRQ3}: now also J4.3 (Pin_3); no longer J4.15 (Pin_15)
- net ~{IRQ4}: now also J4.7 (Pin_7); no longer J4.19 (Pin_19)
- net ~{IRQ5}: now also J4.11 (Pin_11); no longer J4.23 (Pin_23)
- net ~{IRQ6}: now also J4.15 (Pin_15); no longer J4.27 (Pin_27)
- net ~{IRQ7}: now also J4.19 (Pin_19); no longer J4.31 (Pin_31)
- net ~{MEG0}: now also J8.15 (Pin_15), U10.15 (O); no longer J8.3 (Pin_3), U10.22 (O)
- net ~{MEG2}: now also J8.13 (Pin_13), U10.16 (O); no longer J8.5 (Pin_5), U10.21 (O)
- net ~{MEG4}: now also J8.11 (Pin_11), U10.17 (O); no longer J8.6 (Pin_6), U10.20 (O)
- net ~{MEG6}: now also J8.9 (Pin_9), U10.18 (O); no longer J8.8 (Pin_8), U10.19 (O)
- net ~{MEG8}: now also J8.7 (Pin_7), U10.19 (O); no longer U10.18 (O)
- net ~{MEGA}: now also J8.5 (Pin_5), U10.20 (O); no longer U10.17 (O)
- net ~{MEGC}: now also J8.3 (Pin_3), U10.21 (O); no longer U10.16 (O)
- net ~{MEGE}: now also J8.1 (Pin_1), U10.22 (O); no longer U10.15 (O)
- net ~{RAM_OE}: now also J8.17 (Pin_17); no longer J8.9 (Pin_9)
- net ~{WR}: no longer J8.10 (Pin_10)
- no-connect marks 2 -> 1
Other:
- added sheet TurboClock (TurboClock.kicad_sch)
- note added: "2MB ~{CS}"
- note added: "IRQ Priority"
- note added: "IRQ Rewrite"
- note added: "~{VP}*~{E}*A1*A2*A3"
- note removed: "Note: Not subject to ~{VP} Rewrite and associated delay. See 65816 datasheet 2.28"
- note removed: "Note: ~{VP} Rewrite of A1-A4 applies only to low RAM bus. See 65816 datasheet 2.28"
- note removed: "RAM BUS 0 Low 8 MB"
- note removed: "RAM BUS 1 High 8 MB"
- note removed: "Turbo Clock"
- note removed: "Vector Pull Rewrite"
- moved on the sheet: RN1
