File: AronnaxMemory/Serial.kicad_sch (KiCad schematic)
At the start: 1 part, among them X2 28MHz

Commit message: All of it
Parts:
- renumbered X2 to X1
Changed lines of the file:
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@@
 		(on_board yes)
 		(dnp no)
-		(property "Reference" "X2"
+		(property "Reference" "X1"
 			(at 63.5 66.04 0)
 			(effects
@@
 			(project "AronnaxMemory"
 				(path "/f3290a4d-b1bc-4282-9c8a-cd936fe74ce9/e061d0f6-d3bd-4b6b-b744-11d31e8b3e33"
-					(reference "X2")
+					(reference "X1")
 					(unit 1)
 				)
