File: AronnaxMemory/Clock.kicad_sch (KiCad schematic)
At the start: 9 parts, among them J11 Conn_02x18_Odd_Even, J4 Conn_02x40_Odd_Even, J5 GF IO Module, U13 74HC74, U14 74AHCT32, U15 74HC74, U16 74AHCT245, X2 16MHz

Commit message: All of it p2
Parts:
- removed J11: Conn_02x18_Odd_Even, Connector_PinHeader_2.54mm:PinHeader_2x18_P2.54mm_Vertical, symbol Connector_Generic:Conn_02x18_Odd_Even
- removed J4: Conn_02x40_Odd_Even, Connector_PinHeader_2.54mm:PinHeader_2x40_P2.54mm_Vertical, symbol Connector_Generic:Conn_02x40_Odd_Even
- removed J5: GF IO Module, Connector_PinHeader_2.54mm:PinHeader_2x18_P2.54mm_Vertical, symbol Connector_Generic:Conn_02x18_Odd_Even
- removed U16: 74AHCT245, Package_DIP:DIP-20_W7.62mm_Socket, symbol AronnaxLibrary:74AHCT245
Other:
- note removed: "Do not solder the ground side when using the PCB on a breadboard"
- note removed: "OUTPUT"
- moved on the sheet: R13, U13B, U14A, U14B, U14C, U14D, U14E, U15A, U15B, U15C, X2
