File: AronnaxMemory/AronnaxMemory.kicad_sch (KiCad schematic)
At the start: 35 parts, among them J1 Barrel_Jack_Switch, J2 Conn_02x40_Odd_Even, J3 Conn_02x18_Odd_Even, J5 I/O, J8 Conn_02x40_Odd_Even, U1 W65C22SxP, U10 ATF22V10, U4 ATF22V10, U5 74LS348, U6 AS6C4008-55PCN, U7 AT28C256-15PU, U8 ATF22V10, U9 ATF22V10

Commit message: All of it
Parts:
- removed J5: I/O, Connector_PinHeader_2.54mm:PinHeader_2x09_P2.54mm_Vertical, symbol Connector_Generic:Conn_02x09_Odd_Even
- removed U1: W65C22SxP, Package_LCC:PLCC-44_THT-Socket, symbol BB816:W65C22SxP_PLC44
- removed U6: AS6C4008-55PCN, Package_DIP:DIP-32_W15.24mm_Socket, symbol Memory_RAM:AS6C4008-55PCN
- removed U7: AT28C256-15PU, Package_LCC:PLCC-32_THT-Socket, symbol Memory_EEPROM:28C256
- removed U8: ATF22V10, Package_DIP:DIP-24_W7.62mm_Socket, symbol my:ATF22V10
- added C11, C12: 100nF, Capacitor_THT:C_Disc_D3.4mm_W2.1mm_P2.50mm, symbol Device:C
- added J12: Conn_02x08_Odd_Even, Connector_PinHeader_2.54mm:PinHeader_2x08_P2.54mm_Vertical, symbol Connector_Generic:Conn_02x08_Odd_Even
- added J13: Conn_02x18_Odd_Even, PCB_Edge_Connectors:PCB_Edge_36pin, symbol Connector_Generic:Conn_02x18_Odd_Even
- added J9: VP A1-A4, Connector_PinHeader_2.54mm:PinHeader_2x04_P2.54mm_Vertical, symbol Connector_Generic:Conn_02x04_Odd_Even
- J8: value Conn_02x40_Odd_Even -> Conn_02x10_Odd_Even; footprint Connector_PinHeader_2.54mm:PinHeader_2x40_P2.54mm_Vertical -> Connector_PinHeader_2.54mm:PinHeader_2x10_P2.54mm_Vertical; symbol Connector_Generic:Conn_02x40_Odd_Even -> Connector_Generic:Conn_02x10_Odd_Even
Connections:
- net A1: now also J3.17 (Pin_17), U4.5 (I); no longer U4.2 (I)
- net A2: now also J3.15 (Pin_15), U4.4 (I); no longer U4.3 (I)
- net A3: now also J3.13 (Pin_13), U4.3 (I); no longer U4.4 (I)
- net A4: now also J3.11 (Pin_11), U4.2 (I); no longer U4.5 (I)
- net A7: now also U9.11 (I)
- net AA1: now also J9.7 (Pin_7); no longer J3.17 (Pin_17), J8.4 (Pin_4)
- net AA2: now also J9.5 (Pin_5); no longer J3.15 (Pin_15), J8.6 (Pin_6)
- net AA3: now also J9.3 (Pin_3); no longer J3.13 (Pin_13), J8.8 (Pin_8)
- net AA4: now also J9.1 (Pin_1); no longer J3.11 (Pin_11), J8.10 (Pin_10)
- net E: now also U9.1 (CLK); no longer U9.11 (I)
- net GND: now also C11.2, C12.2, J12.1 (Pin_1), J12.11 (Pin_11), J12.13 (Pin_13), J12.15 (Pin_15), J12.3 (Pin_3), J12.5 (Pin_5), J12.7 (Pin_7), J12.9 (Pin_9), J9.2 (Pin_2), J9.4 (Pin_4), J9.6 (Pin_6), J9.8 (Pin_8); no longer J8.21 (Pin_21), J8.23 (Pin_23), J8.25 (Pin_25), J8.27 (Pin_27), J8.29 (Pin_29), J8.31 (Pin_31), J8.33 (Pin_33), J8.35 (Pin_35), J8.37 (Pin_37), J8.39 (Pin_39), J8.41 (Pin_41), J8.43 (Pin_43), J8.45 (Pin_45), J8.47 (Pin_47), J8.49 (Pin_49), J8.51 (Pin_51), J8.53 (Pin_53), J8.55 (Pin_55), J8.57 (Pin_57), J8.59 (Pin_59), J8.61 (Pin_61), J8.63 (Pin_63), J8.65 (Pin_65), J8.67 (Pin_67), J8.69 (Pin_69), J8.71 (Pin_71), J8.73 (Pin_73), J8.75 (Pin_75), J8.77 (Pin_77), J8.79 (Pin_79)
- net VCC: now also C11.1, C12.1; no longer J8.50 (Pin_50), J8.52 (Pin_52)
- net ~{IRQ0}: now also J12.16 (Pin_16)
- net ~{IRQ1}: now also J12.14 (Pin_14)
- net ~{IRQ2}: now also J12.12 (Pin_12)
- net ~{IRQ3}: now also J12.10 (Pin_10)
- net ~{IRQ4}: now also J12.8 (Pin_8)
- net ~{IRQ5}: now also J12.6 (Pin_6)
- net ~{IRQ6}: now also J12.4 (Pin_4)
- net ~{IRQ7}: now also J12.2 (Pin_2); no longer J8.2 (Pin_2)
- net ~{IRQ}: now also J13.33 (Pin_33)
- net ~{MEG0}: now also J8.4 (Pin_4); no longer J8.14 (Pin_14)
- net ~{MEG2}: now also J8.6 (Pin_6); no longer J8.16 (Pin_16)
- net ~{MEG4}: now also J8.8 (Pin_8); no longer J8.18 (Pin_18)
- net ~{MEG6}: now also J8.10 (Pin_10); no longer J8.20 (Pin_20)
- net ~{MEG8}: now also J8.14 (Pin_14); no longer J8.22 (Pin_22)
- net ~{MEGA}: now also J8.16 (Pin_16); no longer J8.24 (Pin_24)
- net ~{MEGC}: now also J8.18 (Pin_18); no longer J8.26 (Pin_26)
- net ~{MEGE}: now also J8.20 (Pin_20); no longer J8.28 (Pin_28)
- net ~{NMI}: now also J13.32 (Pin_32)
- net ~{RAM_OE}: now also J8.2 (Pin_2)
- net ~{IRQV}: now reaches D3.1 (K), R14.2, U5.14 (GS)
- removed net ACIA0_Rx: J8.76 (Pin_76)
- removed net ACIA0_Tx: J8.74 (Pin_74)
- removed net ACIA1_Rx: J8.80 (Pin_80)
- removed net ACIA1_Tx: J8.78 (Pin_78)
- removed net CA1: J8.56 (Pin_56)
- removed net CA2: J8.54 (Pin_54)
- removed net CB1: J8.32 (Pin_32)
- removed net CB2: J8.30 (Pin_30)
- removed net PA0: J8.72 (Pin_72)
- removed net PA1: J8.70 (Pin_70)
- removed net PA2: J8.68 (Pin_68)
- removed net PA3: J8.66 (Pin_66)
- removed net PA4: J8.64 (Pin_64)
- removed net PA5: J8.62 (Pin_62)
- removed net PA6: J8.60 (Pin_60)
- removed net PA7: J8.58 (Pin_58)
- removed net PB0: J8.48 (Pin_48)
- removed net PB1: J8.46 (Pin_46)
- removed net PB2: J8.44 (Pin_44)
- removed net PB3: J8.42 (Pin_42)
- removed net PB4: J8.40 (Pin_40)
- removed net PB5: J8.38 (Pin_38)
- removed net PB6: J8.36 (Pin_36)
- removed net PB7: J8.34 (Pin_34)
- new net GND2: J13.13 (Pin_13), J13.19 (Pin_19), J13.25 (Pin_25), J13.31 (Pin_31), J13.7 (Pin_7)
- new net IOWAIT: J13.34 (Pin_34)
- new net VDD: J13.29 (Pin_29), J13.8 (Pin_8)
- new net XA0: J13.30 (Pin_30)
- new net XA1: J13.27 (Pin_27)
- new net XA10: J13.6 (Pin_6)
- new net XA11: J13.5 (Pin_5)
- new net XA12: J13.4 (Pin_4)
- new net XA13: J13.3 (Pin_3)
- new net XA14: J13.1 (Pin_1)
- new net XA2: J13.28 (Pin_28)
- new net XA3: J13.26 (Pin_26)
- new net XA4: J13.23 (Pin_23)
- new net XA5: J13.24 (Pin_24)
- new net XA6: J13.22 (Pin_22)
- new net XA7: J13.21 (Pin_21)
- new net XA8: J13.10 (Pin_10)
- new net XA9: J13.9 (Pin_9)
- new net XD0: J13.20 (Pin_20)
- new net XD1: J13.18 (Pin_18)
- new net XD2: J13.17 (Pin_17)
- new net XD3: J13.16 (Pin_16)
- new net XD4: J13.15 (Pin_15)
- new net XD5: J13.14 (Pin_14)
- new net XD6: J13.12 (Pin_12)
- new net XD7: J13.11 (Pin_11)
- new net XR~{W}: J13.2 (Pin_2)
- new net ~{IOREADY}: J13.35 (Pin_35)
- new net ~{RESET}: J13.36 (Pin_36)
Other:
- added sheet Clock (Clock.kicad_sch)
- added sheet IO_SEL (IO_SEL.kicad_sch)
- added sheet RAM (RAM.kicad_sch)
- added sheet ROM (ROM.kicad_sch)
- added sheet VIA (VIA.kicad_sch)
- note added: "IRQ"
- note removed: "32KB ROM 0x008000 0x00FFFF"
- note removed: "512KB RAM 0x000000 0x07FFFF"
- note removed: "I/O Bus"
- note removed: "I/O Select"
- note removed: "Memory 512KB RAM + 32KB ROM"
- note removed: "System VIA ~{IO_0} ~{IRQ0}"
- moved on the sheet: C1, C10, C2, C3, C4, C5, C6, C7, C8, C9, RN1

Commit message: All of it p2
Parts:
- removed C10, C11, C12, C8, C9: 100nF, Capacitor_THT:C_Disc_D3.4mm_W2.1mm_P2.50mm, symbol Device:C
- removed J13: Conn_02x18_Odd_Even, PCB_Edge_Connectors:PCB_Edge_36pin, symbol Connector_Generic:Conn_02x18_Odd_Even
- added J11: Conn_02x18_Odd_Even, PCB_Edge_Connectors:PCB_Edge_36pin, symbol Connector_Generic:Conn_02x18_Odd_Even
- added R13: 3.3k, Resistor_THT:R_Axial_DIN0207_L6.3mm_D2.5mm_P7.62mm_Horizontal, symbol Device:R_Small
- added U13, U5: 74HC74, Package_DIP:DIP-14_W7.62mm, symbol 74xx:74LS74
- added U4: 74AHCT32, Package_DIP:DIP-14_W7.62mm_Socket, symbol AronnaxLibrary:74AHCT32
- added X1: 16MHz, Oscillator:Oscillator_DIP-8, symbol Oscillator:CXO_DIP8
- J12: value Conn_02x08_Odd_Even -> IRQ In
- J8: value Conn_02x10_Odd_Even -> 2MB Select; footprint Connector_PinHeader_2.54mm:PinHeader_2x10_P2.54mm_Vertical -> Connector_PinHeader_2.54mm:PinHeader_2x09_P2.54mm_Vertical; symbol Connector_Generic:Conn_02x10_Odd_Even -> Connector_Generic:Conn_02x09_Odd_Even
- renumbered U9 to U2, U10 to U3, U5 to U6, U4 to U7
Connections:
- net ~{RAM_RD} is gone; now on net ~{RAM_OE}: U3.23 (O)
- net A0: now also J11.30 (Pin_30)
- net A1: now also J11.27 (Pin_27)
- net A10: now also J11.6 (Pin_6)
- net A11: now also J11.5 (Pin_5)
- net A12: now also J11.4 (Pin_4)
- net A13: now also J11.3 (Pin_3)
- net A14: now also J11.1 (Pin_1)
- net A2: now also J11.28 (Pin_28)
- net A3: now also J11.26 (Pin_26)
- net A4: now also J11.23 (Pin_23)
- net A5: now also J11.24 (Pin_24)
- net A6: now also J11.22 (Pin_22)
- net A7: now also J11.21 (Pin_21)
- net A8: now also J11.10 (Pin_10)
- net A9: now also J11.9 (Pin_9)
- net CLK_SRC: now also U4.6
- net D0: now also J11.20 (Pin_20)
- net D1: now also J11.18 (Pin_18)
- net D2: now also J11.17 (Pin_17)
- net D3: now also J11.16 (Pin_16)
- net D4: now also J11.15 (Pin_15)
- net D5: now also J11.14 (Pin_14)
- net D6: now also J11.12 (Pin_12)
- net D7: now also J11.11 (Pin_11)
- net GND: now also U4.1, U4.13, U4.2, U4.7 (GND), U4.9, U5.7 (GND), X1.4 (GND); no longer J8.19 (Pin_19), J9.2 (Pin_2), J9.4 (Pin_4), J9.6 (Pin_6), J9.8 (Pin_8)
- net GND2: now also J11.13 (Pin_13), J11.19 (Pin_19), J11.25 (Pin_25), J11.31 (Pin_31), J11.7 (Pin_7)
- net IOWAIT: now also J11.34 (Pin_34), U4.4, U5.4 (~{S}), U5.9 (Q)
- net R~{W}: now also J11.2 (Pin_2)
- net VCC: now also R13.1, U13.10 (~{S}), U13.13 (~{R}), U4.14 (VCC), U5.1 (~{R}), U5.10 (~{S}), U5.14 (VCC), X1.8 (Vcc)
- net VDD: now also J11.29 (Pin_29), J11.8 (Pin_8)
- net ~{CLK_EN}: now also R13.2; no longer U2.20 (O)
- net ~{IOREADY}: now also J11.35 (Pin_35), U5.2 (D)
- net ~{IRQ}: now also J11.33 (Pin_33)
- net ~{MEG0}: now also J8.2 (Pin_2); no longer J8.4 (Pin_4)
- net ~{MEG2}: now also J8.4 (Pin_4); no longer J8.6 (Pin_6)
- net ~{MEG4}: now also J8.6 (Pin_6); no longer J8.8 (Pin_8)
- net ~{MEG6}: now also J8.8 (Pin_8); no longer J8.10 (Pin_10)
- net ~{MEG8}: now also J8.10 (Pin_10); no longer J8.14 (Pin_14)
- net ~{MEGA}: now also J8.12 (Pin_12); no longer J8.16 (Pin_16)
- net ~{MEGC}: now also J8.14 (Pin_14); no longer J8.18 (Pin_18)
- net ~{MEGE}: now also J8.16 (Pin_16); no longer J8.20 (Pin_20)
- net ~{NMI}: now also J11.32 (Pin_32)
- net ~{RAM_OE}: now also J8.18 (Pin_18); no longer J8.12 (Pin_12), J8.2 (Pin_2)
- net ~{RESET}: now also J11.36 (Pin_36)
- net BE: no longer names the net of J2.25 (Pin_25)
- net CLK: no longer names the net of J2.15 (Pin_15)
- net M: no longer names the net of J2.45 (Pin_45)
- net RDY_IN: no longer names the net of J2.27 (Pin_27)
- net RST: no longer names the net of J2.9 (Pin_9)
- net SYNC: no longer names the net of J2.31 (Pin_31)
- net VA: no longer names the net of J2.33 (Pin_33)
- net X: no longer names the net of J2.47 (Pin_47)
- net ~{ABORT}: no longer names the net of J2.23 (Pin_23)
- net ~{CLK}: no longer names the net of J2.17 (Pin_17)
- net ~{ML}: no longer names the net of J2.51 (Pin_51)
- net ~{MR}⎒: no longer names the net of J2.5 (Pin_5)
- net ~{WAI}: no longer names the net of J2.29 (Pin_29)
- new net: J9.2 (Pin_2), J9.4 (Pin_4), J9.6 (Pin_6), J9.8 (Pin_8)
- new net: U4.10, U4.11
- new net: U13.12 (D), U13.8 (~{Q})
- new net 16MHz: U13.11 (C), X1.5 (OUT)
- new net 8MHz: U13.9 (Q), U4.12, U4.5
- new net DCLK: U4.8, U5.11 (C), U5.3 (C)
- new net STRETCH: U5.12 (D)
- new net ~{RDYRESET}: U5.13 (~{R}), U5.5 (Q)
- no-connect marks 1 -> 19
Other:
- removed sheet Clock
- removed sheet IO_SEL
- removed sheet RAM
- removed sheet ROM
- removed sheet Serial
- removed sheet VIA
- note added: "2MB Select"
- note added: "After M. Adrien Kohlbecker (BB816 Breakout v.A27) After Mr. George Foot (Fast PDIP 6502)"
- note added: "Application Note ~{CLK_EN} is pulled high to disable BB816 clock Do not install R11 on BB816 rev. A27"
- note added: "BB816 A27 / Fast PDIP 6502 I/O Adapter with IRQ Vector Pull Rewrite"
- note added: "GFoot 6502 I/O Module"
- note removed: "2MB Boundaries"
- note removed: "After M. Adrien Kohlbecker (BB816 Breakout v.A27)"
- note removed: "BB816 Programmable System Controller"
- note removed: "Bank Address"
- note removed: "IRQ"
- moved on the sheet: C1, C2, C21, C22, C3, C4, C5, C6, C7, D1, D3, J1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

Commit message: All of it.
Parts:
- removed D3: 1N4148, Diode_THT:D_DO-35_SOD27_P7.62mm_Horizontal, symbol Diode:1N4148
- removed R14: 10K, Resistor_THT:R_Axial_DIN0207_L6.3mm_D2.5mm_P7.62mm_Horizontal, symbol Device:R
- added D4: 1N4148, Diode_THT:D_DO-35_SOD27_P7.62mm_Horizontal, symbol Diode:1N4148
- added R15: 10K, Resistor_THT:R_Axial_DIN0207_L6.3mm_D2.5mm_P7.62mm_Horizontal, symbol Device:R
Connections:
- net GND2 is gone; now on net GND: J11.13 (Pin_13), J11.19 (Pin_19), J11.25 (Pin_25), J11.31 (Pin_31), J11.7 (Pin_7)
- net VDD is gone; now on net VCC: J11.29 (Pin_29), J11.8 (Pin_8)
- net ~{IRQV} is gone; now on net ~{IRQ_VALID}: U6.14 (GS)
- net E: now also U7.11 (I)
- net VCC: now also R15.1
- net ~{IRQ}: now also D4.2 (A); no longer U7.16 (O)
- net ~{ROM_OE}: no longer U2.22 (O)
- net ~{IRQ_ASSERT}: now reaches U7.23 (O)
- net ~{IRQ_ASSERT}: now also D4.1 (K), R15.2
- net ~{IRQ_VALID}: now reaches U7.6 (I)
- net ~{RAM_OE} renamed I/O
- net I/O: now also U2.22 (O); no longer U2.21 (O)
Other:
- note added: "Application Note Do not install IRQ diodes in George Foot Fast I/O Module."
- note added: "Clock"
- note added: "Fast PDIP 6502 I/O Module"
- note added: "IRQ Vector Rewrite"
- note removed: "GFoot 6502 I/O Module"
- note removed: "Reversed? Swap pins in symbol?"
- moved on the sheet: J11, R3, R4, R5

Commit message: Before replacing 22V10 with 4 bit adder
Parts:
- added C10, C8, C9: 100nF, Capacitor_THT:C_Disc_D3.4mm_W2.1mm_P2.50mm, symbol Device:C
- added JP1, JP2, JP3, JP4: Jumper3_254mm, Jumper3_254mm:Jumper3_254mm, symbol Jumper3_254mm:Jumper3_254mm
- added U10, U9: AS6C4008-55PCN, Package_DIP:DIP-32_W15.24mm_Socket, symbol Memory_RAM:AS6C4008-55PCN
- added unit 3 of U8
- added unit 1 of U8
- J8: value 2MB Select -> RAM Select
- renumbered R5 to R1, R4 to R2, R6 to R4, R15 to R5, R13 to R6, U13 to U8
Connections:
- net ~{ROM_OE} is gone; now on net A16: U3.11 (I)
- net ~{RST} is gone; now on net ~{RESET}: J2.7 (Pin_7)
- net A0: now also U10.12 (A0), U9.12 (A0)
- net A1: now also JP1.3 (B)
- net A10: now also U10.23 (A10), U9.23 (A10)
- net A11: now also U10.25 (A11), U9.25 (A11)
- net A12: now also U10.4 (A12), U9.4 (A12)
- net A13: now also U10.28 (A13), U9.28 (A13)
- net A14: now also U10.3 (A14), U9.3 (A14)
- net A15: now also U10.31 (A15), U9.31 (A15)
- net A16: now also U10.2 (A16), U9.2 (A16); no longer U3.9 (I)
- net A17: now also U3.10 (I), U10.30 (A17), U9.30 (A17); no longer U3.8 (I)
- net A18: now also U3.9 (I), U10.1 (A18), U9.1 (A18); no longer U3.7 (I)
- net A19: now also U3.8 (I); no longer U3.6 (I)
- net A2: now also JP2.3 (B)
- net A20: now also U3.7 (I); no longer U3.5 (I)
- net A21: now also U3.6 (I); no longer U3.4 (I)
- net A22: now also U3.5 (I); no longer U3.3 (I)
- net A23: now also U3.4 (I); no longer U3.2 (I)
- net A3: now also JP3.3 (B)
- net A4: now also JP4.3 (B)
- net A5: now also U10.7 (A5), U9.7 (A5)
- net A6: now also U10.6 (A6), U9.6 (A6)
- net A7: now also U10.5 (A7), U9.5 (A7)
- net A8: now also U10.27 (A8), U9.27 (A8)
- net A9: now also U10.26 (A9), U9.26 (A9)
- net AA1: now also J9.1 (Pin_1), U7.20 (O), JP1.1 (A); no longer J9.7 (Pin_7), U7.17 (O)
- net AA2: now also J9.3 (Pin_3), U7.19 (O), JP2.1 (A); no longer J9.5 (Pin_5), U7.18 (O)
- net AA3: now also J9.5 (Pin_5), U7.18 (O), JP3.1 (A); no longer J9.3 (Pin_3), U7.19 (O)
- net AA4: now also J9.7 (Pin_7), U7.17 (O), JP4.1 (A); no longer J9.1 (Pin_1), U7.20 (O)
- net D0: now also U10.13 (DQ0), U9.13 (DQ0)
- net D1: now also U10.14 (DQ1), U9.14 (DQ1)
- net D2: now also U10.15 (DQ2), U9.15 (DQ2)
- net D3: now also U10.17 (DQ3), U9.17 (DQ3)
- net D4: now also U10.18 (DQ4), U9.18 (DQ4)
- net D5: now also U10.19 (DQ5), U9.19 (DQ5)
- net D6: now also U10.20 (DQ6), U9.20 (DQ6)
- net D7: now also U10.21 (DQ7), U9.21 (DQ7)
- net E: no longer U7.11 (I)
- net GND: now also C10.2, C8.2, C9.2, U10.16 (VSS), U8.2 (D), U8.3 (C), U8.7 (GND), U9.16 (VSS)
- net VCC: now also C10.1, C8.1, C9.1, U10.32 (VCC), U8.1 (~{R}), U8.14 (VCC), U8.4 (~{S}), U9.32 (VCC)
- net ~{IRQ_VALID}: now also D4.1 (K), R5.2; no longer U7.6 (I)
- net ~{NMI}: no longer U7.21 (O)
- net ~{RD}: now also U3.3 (I); no longer U3.1 (CLK)
- net ~{VP}: now also U2.13 (I); no longer U7.10 (I)
- net ~{WR}: now also U10.29 (WE#), U9.29 (WE#)
- net I/O renamed ~{RAM_OE}
- net ~{RAM_OE}: now also U10.24 (OE#), U9.24 (OE#); no longer U2.22 (O)
- net STRETCH renamed IO_AREA
- net IO_AREA: now also U2.23 (O), U3.2 (I)
- removed net ~{IRQ_ASSERT}: D4.1 (K), R5.2, U7.23 (O)
- removed net ~{I/O}: U2.23 (O), U3.10 (I)
- net ~{MEG0} renamed ~{RAM_0}
- net ~{RAM_0}: now also U9.22 (CE#)
- net ~{MEG2} renamed ~{RAM_1}
- net ~{RAM_1}: now also U10.22 (CE#)
- net ~{MEG4} renamed ~{RAM_2}
- net ~{MEG6} renamed ~{RAM_3}
- net ~{MEG8} renamed ~{RAM_4}
- net ~{MEGA} renamed ~{RAM_5}
- net ~{MEGC} renamed ~{RAM_6}
- net ~{MEGE} renamed ~{RAM_7}
- new net BA1: JP1.2 (C), U10.11 (A1), U9.11 (A1)
- new net BA2: JP2.2 (C), U10.10 (A2), U9.10 (A2)
- new net BA3: JP3.2 (C), U10.9 (A3), U9.9 (A3)
- new net BA4: JP4.2 (C), U10.8 (A4), U9.8 (A4)
- new net ~{VP_REWRITE}: U2.22 (O), U7.10 (I)
- no-connect marks 19 -> 20
Other:
- note added: "512KB RAM 0x000000 0x07FFFF"
- note added: "512KB RAM 0x080000 0x0FFFFF"
- note added: "A1-4 Bypass"
- note added: "I/O Area"
- note added: "I/O Module"
- note added: "RAM"
- note added: "RAM ~{CS}"
- note added: "after Adrien Kohlbecker (BB816 Breakout v.A27) after George Foot (Fast PDIP 6502 I/O Module)"
- note removed: "2MB Select"
- note removed: "Address Decode - IRQ Vector Pull Rewrite - Native Mode Turbo Clock - 512KB RAM - 32KB ROM CPLDs allow fine grain tuning. This design can implement the memory map of BigDumbMonkey's POC 1 design. This design implements section 2.28 of the 65816 datasheet. Shadow RAM allows banking out slower EEPROM once startup is complete."
- note removed: "After M. Adrien Kohlbecker (BB816 Breakout v.A27) After Mr. George Foot (Fast PDIP 6502)"
- note removed: "Fast PDIP 6502 I/O Module"
- note removed: "I/O+ROM Area"
- moved on the sheet: C1, C2, C21, C22, C3, C4, C5, C6, C7, D1, D4, J1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

Commit message: Gettin ready to publish
Parts:
- added C11, C12: 100nF, Capacitor_THT:C_Disc_D3.4mm_W2.1mm_P2.50mm, symbol Device:C
- added U11, U12: AS6C4008-55PCN, Package_DIP:DIP-32_W15.24mm_Socket, symbol Memory_RAM:AS6C4008-55PCN
Connections:
- net A17 is gone; now on net A16: J2.65 (Pin_65), U10.30 (A17), U3.10 (I), U9.30 (A17)
- net A18 is gone; now on net A16: J2.63 (Pin_63), U10.1 (A18), U3.9 (I), U9.1 (A18)
- net A19 is gone; now on net A16: J2.61 (Pin_61), U3.8 (I)
- net A20 is gone; now on net A16: J2.59 (Pin_59), U3.7 (I)
- net A21 is gone; now on net A16: J2.57 (Pin_57), U3.6 (I)
- net A22 is gone; now on net A16: J2.55 (Pin_55), U3.5 (I)
- net A23 is gone; now on net A16: J2.53 (Pin_53), U3.4 (I)
- net A0: now also U11.12 (A0), U12.12 (A0)
- net A10: now also U2.7 (I), U11.23 (A10), U12.23 (A10); no longer U2.8 (I)
- net A11: now also U2.6 (I), U11.25 (A11), U12.25 (A11); no longer U2.7 (I)
- net A12: now also U2.5 (I), U11.4 (A12), U12.4 (A12); no longer U2.6 (I)
- net A13: now also U2.4 (I), U11.28 (A13), U12.28 (A13); no longer U2.5 (I)
- net A14: now also U2.3 (I), U11.3 (A14), U12.3 (A14); no longer U2.4 (I)
- net A15: now also U2.2 (I), U11.31 (A15), U12.31 (A15); no longer U2.3 (I)
- net A16: now also U2.22 (O), U7.6 (I), U7.8 (I), U7.9 (I), U11.1 (A18), U11.2 (A16), U11.30 (A17), U12.1 (A18), U12.2 (A16), U12.30 (A17)
- net A5: now also U11.7 (A5), U12.7 (A5)
- net A6: now also U11.6 (A6), U12.6 (A6)
- net A7: now also U2.10 (I), U11.5 (A7), U12.5 (A7); no longer U2.11 (I)
- net A8: now also U2.9 (I), U11.27 (A8), U12.27 (A8); no longer U2.10 (I)
- net A9: now also U2.8 (I), U11.26 (A9), U12.26 (A9); no longer U2.9 (I)
- net AA2: now also U7.21 (O); no longer U7.19 (O)
- net AA3: now also U7.22 (O); no longer U7.18 (O)
- net AA4: now also U7.23 (O); no longer U7.17 (O)
- net ADDEND_AA1: now also U7.13 (I); no longer U7.7 (I)
- net ADDEND_AA2: now also U7.14 (O); no longer U7.8 (I)
- net ADDEND_AA3: now also U7.15 (O); no longer U7.9 (I)
- net BA1: now also U11.11 (A1), U12.11 (A1)
- net BA2: now also U11.10 (A2), U12.10 (A2)
- net BA3: now also U11.9 (A3), U12.9 (A3)
- net BA4: now also U11.8 (A4), U12.8 (A4)
- net D0: now also U11.13 (DQ0), U12.13 (DQ0)
- net D1: now also U11.14 (DQ1), U12.14 (DQ1)
- net D2: now also U11.15 (DQ2), U12.15 (DQ2)
- net D3: now also U11.17 (DQ3), U12.17 (DQ3)
- net D4: now also U11.18 (DQ4), U12.18 (DQ4)
- net D5: now also U11.19 (DQ5), U12.19 (DQ5)
- net D6: now also U11.20 (DQ6), U12.20 (DQ6)
- net D7: now also U11.21 (DQ7), U12.21 (DQ7)
- net E: now also U2.14 (O); no longer U2.1 (CLK)
- net GND: now also J9.2 (Pin_2), J9.4 (Pin_4), J9.6 (Pin_6), J9.8 (Pin_8), U2.1 (CLK), U3.1 (CLK), U3.13 (I), U7.1 (CLK), U7.10 (I), U7.11 (I), C11.2, C12.2, U11.16 (VSS), U12.16 (VSS)
- net VCC: now also C11.1, C12.1, U11.32 (VCC), U12.32 (VCC)
- net ~{BANK0}: now also U2.11 (I); no longer U2.2 (I)
- net ~{RAM_0}: now also U7.19 (O); no longer J8.2 (Pin_2), U3.15 (O)
- net ~{RAM_1}: now also U7.18 (O); no longer J8.4 (Pin_4), U3.16 (O)
- net ~{RAM_2}: now also U7.17 (O), U11.22 (CE#); no longer J8.6 (Pin_6), U3.17 (O)
- net ~{RAM_3}: now also U7.16 (O), U12.22 (CE#); no longer J8.8 (Pin_8), U3.18 (O)
- net ~{RAM_OE}: now also U11.24 (OE#), U12.24 (OE#)
- net ~{WR}: now also U11.29 (WE#), U12.29 (WE#)
- net ~{RAM_4} renamed ~{2M_4}
- net ~{RAM_5} renamed ~{2M_5}
- net ~{RAM_6} renamed ~{2M_6}
- net ~{RAM_7} renamed ~{2M_7}
- removed net ~{VP_REWRITE}: U2.22 (O), U7.10 (I)
- new net ~{2M_0}: J8.2 (Pin_2), U3.15 (O), U7.7 (I)
- new net ~{2M_1}: J8.4 (Pin_4), U3.16 (O)
- new net ~{2M_2}: J8.6 (Pin_6), U3.17 (O)
- new net ~{2M_3}: J8.8 (Pin_8), U3.18 (O)
- no-connect marks 20 -> 28
Other:
- note added: "2M ~{CS}"
- note added: "512KB RAM 0x100000 0x17FFFF"
- note added: "512KB RAM 0x180000 0x1FFFFF"
- note added: "BB816 Rev.A27"
- note added: "GFoot I/O"
- note added: "IRQ Vector Rewrite + 512KB ~{CS}"
- note removed: "A1-A4 Offset"
- note removed: "BB816"
- note removed: "I/O Module"
- note removed: "IRQ Rewrite"
- note removed: "IRQ Vector Rewrite"
- note removed: "Native Mode Only See 65816 datasheet section 2.28"
- note removed: "RAM ~{CS}"
- note removed: "~{VP}*~{E}*A1*A2*A3"
- moved on the sheet: C1, C10, C2, C21, C22, C3, C4, C5, C6, C7, C8, C9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
