File: AronnaxMemory/AronnaxMemory.kicad_sch (KiCad schematic)
At the start: 48 parts, among them J1 Barrel_Jack_Switch, J11 Conn_02x18_Odd_Even, J12 IRQ In, J2 Conn_02x40_Odd_Even, J3 Conn_02x18_Odd_Even, J8 RAM Select, J9 VP A1-A4, U10 AS6C4008-55PCN, U11 AS6C4008-55PCN, U12 AS6C4008-55PCN, U2 ATF22V10, U3 ATF22V10, U4 74AHCT32, U5 74HC74, U6 74LS348, U7 ATF22V10, U8 74HC74, U9 AS6C4008-55PCN, X1 16MHz

Commit message: Simplifying Removed VPR
Parts:
- removed C6, C7: 100nF, Capacitor_THT:C_Disc_D3.4mm_W2.1mm_P2.50mm, symbol Device:C
- removed D4: 1N4148, Diode_THT:D_DO-35_SOD27_P7.62mm_Horizontal, symbol Diode:1N4148
- removed J12: IRQ In, Connector_PinHeader_2.54mm:PinHeader_2x08_P2.54mm_Vertical, symbol Connector_Generic:Conn_02x08_Odd_Even
- removed R1, R2, R3, R5: 10K, Resistor_THT:R_Axial_DIN0207_L6.3mm_D2.5mm_P7.62mm_Horizontal, symbol Device:R
- removed RN1: 100k, Resistor_THT:R_Array_SIP9, symbol Device:R_Network08
- removed U6: 74LS348, Package_DIP:DIP-16_W7.62mm_Socket, symbol 74xx:74LS348
- removed U7: ATF22V10, Package_DIP:DIP-24_W7.62mm_Socket, symbol my:ATF22V10
Connections:
- net ~{2M_0} is gone; now on net ~{RAM_0}: J8.2 (Pin_2), U3.15 (O)
- net ~{2M_1} is gone; now on net ~{RAM_1}: J8.4 (Pin_4), U3.16 (O)
- net ~{2M_2} is gone; now on net ~{RAM_2}: J8.6 (Pin_6), U3.17 (O)
- net ~{2M_3} is gone; now on net ~{RAM_3}: J8.8 (Pin_8), U3.18 (O)
- net A16: no longer J2.53 (Pin_53), J2.55 (Pin_55), J2.57 (Pin_57), J2.59 (Pin_59), J2.61 (Pin_61), J2.63 (Pin_63), J2.65 (Pin_65), U10.1 (A18), U10.30 (A17), U11.1 (A18), U11.30 (A17), U12.1 (A18), U12.30 (A17), U2.22 (O), U3.10 (I), U3.4 (I), U3.5 (I), U3.6 (I), U3.7 (I), U3.8 (I), U3.9 (I), U9.1 (A18), U9.30 (A17)
- net ~{2M_4} renamed ~{RAM_4}
- net ~{2M_5} renamed ~{RAM_5}
- net ~{2M_6} renamed ~{RAM_6}
- net ~{2M_7} renamed ~{RAM_7}
- new net A17: J2.65 (Pin_65), U10.30 (A17), U11.30 (A17), U12.30 (A17), U3.10 (I), U9.30 (A17)
- new net A18: J2.63 (Pin_63), U10.1 (A18), U11.1 (A18), U12.1 (A18), U3.9 (I), U9.1 (A18)
- new net A19: J2.61 (Pin_61), U3.8 (I)
- new net A20: J2.59 (Pin_59), U3.7 (I)
- new net A21: J2.57 (Pin_57), U3.6 (I)
- new net A22: J2.55 (Pin_55), U3.5 (I)
- new net A23: J2.53 (Pin_53), U3.4 (I)
- new net ~{VPR}: U2.22 (O)
Other:
- added sheet VPR (VPR.kicad_sch)
- note added: "RAM ~{CS}"
- note removed: "2M ~{CS}"
- note removed: "Application Note Do not install IRQ diodes in George Foot Fast I/O Module."
- note removed: "IRQ Priority"
- note removed: "IRQ Vector Rewrite + 512KB ~{CS}"
- note removed: "Priority"
- moved on the sheet: C10, C11, C12, C8, C9, U2, U3

Commit message: May 2025
Parts:
- removed C10, C11, C12, C9: 100nF, Capacitor_THT:C_Disc_D3.4mm_W2.1mm_P2.50mm, symbol Device:C
- removed J9: VP A1-A4, Connector_PinHeader_2.54mm:PinHeader_2x04_P2.54mm_Vertical, symbol Connector_Generic:Conn_02x04_Odd_Even
- removed JP1, JP2, JP3, JP4: Jumper3_254mm, Jumper3_254mm:Jumper3_254mm, symbol Jumper3_254mm:Jumper3_254mm
- removed U10, U11, U12, U9: AS6C4008-55PCN, Package_DIP:DIP-32_W15.24mm_Socket, symbol Memory_RAM:AS6C4008-55PCN
- U5: footprint Package_DIP:DIP-14_W7.62mm -> Package_DIP:DIP-14_W7.62mm_Socket
- U6: renamed from U8; footprint Package_DIP:DIP-14_W7.62mm -> Package_DIP:DIP-14_W7.62mm_Socket
- renumbered C8 to C6
Connections:
- net A10: now also U2.8 (I); no longer U2.7 (I)
- net A11: now also U2.7 (I); no longer U2.6 (I)
- net A12: now also U2.6 (I); no longer U2.5 (I)
- net A13: now also U2.5 (I); no longer U2.4 (I)
- net A14: now also U2.4 (I); no longer U2.3 (I)
- net A15: now also U2.3 (I); no longer U2.2 (I)
- net A7: now also U2.11 (I); no longer U2.10 (I)
- net A8: now also U2.10 (I); no longer U2.9 (I)
- net A9: now also U2.9 (I); no longer U2.8 (I)
- net E: now also U3.2 (I); no longer U2.14 (O)
- net GND: now also U3.3 (I); no longer U3.1 (CLK), U3.13 (I)
- net IO_AREA: now also U3.13 (I); no longer U3.2 (I)
- net ~{BANK0}: now also U2.2 (I); no longer U2.11 (I)
- net ~{RD}: now also U3.1 (CLK); no longer U3.3 (I)
- net ~{VP}: no longer U2.13 (I)
- net ~{VPR}: no longer names the net of U2.22 (O)
- no-connect marks 28 -> 30
Other:
- removed sheet VPR
- note removed: "512KB RAM 0x000000 0x07FFFF"
- note removed: "512KB RAM 0x080000 0x0FFFFF"
- note removed: "512KB RAM 0x100000 0x17FFFF"
- note removed: "512KB RAM 0x180000 0x1FFFFF"
- note removed: "A1-4 Bypass"
- note removed: "RAM"
- moved on the sheet: J8
